File: Schema_KICAD/ESE_AL8/ESE_AL8/_autosave-ESE_AL8.kicad_sch (KiCad schematic)
At the start: 21 parts, among them SW101 Reset, U101 STM32G431C6Tx, Y101 16MHz

Commit message: schema_architectural
Other:
- added sheet Schema architectural (schema_architectural.kicad_sch)
Changed lines of the file:
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@@
+	)
+	(sheet
+		(at 184.15 21.59)
+		(size 48.26 30.48)
+		(fields_autoplaced yes)
+		(stroke
+			(width 0.1524)
+			(type solid)
+		)
+		(fill
+			(color 0 0 0 0.0000)
+		)
+		(property "Sheetname" "Schema architectural"
+			(at 184.15 20.8784 0)
+			(effects
+				(font
+					(size 1.27 1.27)
+				)
+				(justify left bottom)
+			)
+		)
+		(property "Sheetfile" "schema_architectural.kicad_sch"
+			(at 184.15 52.6546 0)
+			(effects
+				(font
+					(size 1.27 1.27)
+				)
+				(justify left top)
+			)
+		)
+		(instances
+			(project "ESE_AL8"
+				(path "/c3d0eb52-cd9d-4e69-bcf7-3f0716f715c6"
+					(page "4")
+				)
+			)
+		)
 	)
 	(sheet
