File: Schema_KICAD/ESE_AL8/ESE_AL8/ESE_AL8.kicad_sch (KiCad schematic)
At the start: 21 parts, among them SW101 Reset, U101 STM32G431C6Tx, Y101 16MHz

Commit message: schema_architectural
Other:
- added sheet Schema architectural (schema_architectural.kicad_sch)
Changed lines of the file:
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@@
 		(dnp no)
 		(property "Reference" "C108"
-			(at 82.55 95.25 0)
+			(at 82.042 95.25 0)
 			(effects
 				(font
@@
 		(dnp no)
 		(property "Reference" "D102"
-			(at 54.61 158.75 0)
+			(at 53.848 165.354 0)
 			(effects
 				(font
@@
 		)
 		(property "Value" "LED_USER"
-			(at 60.96 158.75 0)
+			(at 54.61 166.878 0)
 			(effects
 				(font
@@
 				)
 			)
+		)
+	)
+	(sheet
+		(at 184.15 21.59)
+		(size 48.26 30.48)
+		(fields_autoplaced yes)
+		(stroke
+			(width 0.1524)
+			(type solid)
+		)
+		(fill
+			(color 0 0 0 0.0000)
+		)
+		(property "Sheetname" "Schema architectural"
+			(at 184.15 20.8784 0)
+			(effects
+				(font
+					(size 1.27 1.27)
+				)
+				(justify left bottom)
+			)
+		)
+		(property "Sheetfile" "schema_architectural.kicad_sch"
+			(at 184.15 52.6546 0)
+			(effects
+				(font
+					(size 1.27 1.27)
+				)
+				(justify left top)
+			)
+		)
+		(instances
+			(project "ESE_AL8"
+				(path "/c3d0eb52-cd9d-4e69-bcf7-3f0716f715c6"
+					(page "4")
+				)
+			)

Commit message: commit pour 18/09
Parts:
- removed U101: STM32G431C6Tx, Package_QFP:LQFP-48_7x7mm_P0.5mm, symbol MCU_ST_STM32G4:STM32G431C6Tx
- added U101: STM32G431CBUx, Package_DFN_QFN:QFN-48-1EP_7x7mm_P0.5mm_EP5.6x5.6mm, symbol MCU_ST_STM32G4:STM32G431CBUx
- renumbered C110 to C101, C111 to C102, C101 to C103, C108 to C104, C102 to C105, C112 to C106, C109 to C107, C103 to C108, C104 to C109, C105 to C110, C106 to C111, C107 to C112, D102 to D101, D101 to D102, R103 to R101, R101 to R103
Connections:
- net +3.3V: now also U101.1 (VBAT), U101.23 (VDD), U101.35 (VDD), U101.48 (VDD)
- net GND: now also U101.49 (VSS)
- net NRST: now also U101.7 (PG10)
- net OSC_IN: now also U101.5 (PF0)
- net OSC_OUT: now also U101.6 (PF1)
- net VREF+: now also U101.20 (VREF+), U101.21 (VDDA)

Commit message: commit 18/09/24 18:10
Parts:
- R103: value 80 -> 20
Changed lines of the file:
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@@
 			)
 		)
-		(property "Value" "80"
+		(property "Value" "20"
 			(at 88.138 132.08 0)
 			(effects

Commit message: LE 25 /09/2024 10:31
Parts:
- removed C101: 100n, Capacitor_SMD:C_0603_1608Metric_Pad1.08x0.95mm_HandSolder, symbol Device:C_Small
- removed D101: LED_USER, LED_SMD:LED_0603_1608Metric_Pad1.05x0.95mm_HandSolder, symbol Device:LED
- removed R101: 680, Resistor_SMD:R_0603_1608Metric_Pad0.98x0.95mm_HandSolder, symbol Device:R_Small
- removed SW101: Reset, Button_Switch_THT:SW_PUSH_6mm_H4.3mm, symbol Switch:SW_Push
- added H101, H102, H103, H104: MountingHole_Pad, MountingHole:MountingHole_3.2mm_M3_Pad_Via, symbol Mechanical:MountingHole_Pad
- added J101: ECRAN, Connector_PinSocket_2.54mm:PinSocket_1x04_P2.54mm_Vertical, symbol Connector:Screw_Terminal_01x04
- added J102: GPIO, Connector_PinSocket_2.54mm:PinSocket_1x03_P2.54mm_Vertical, symbol Connector:Screw_Terminal_01x03
- C101: renamed from C102; footprint Capacitor_SMD:C_0603_1608Metric_Pad1.08x0.95mm_HandSolder -> Capacitor_SMD:C_0402_1005Metric_Pad0.74x0.62mm_HandSolder
- C103: renamed from C105; footprint Capacitor_SMD:C_0603_1608Metric_Pad1.08x0.95mm_HandSolder -> Capacitor_SMD:C_0402_1005Metric_Pad0.74x0.62mm_HandSolder
- C104: renamed from C106; footprint Capacitor_SMD:C_0603_1608Metric_Pad1.08x0.95mm_HandSolder -> Capacitor_SMD:C_0402_1005Metric_Pad0.74x0.62mm_HandSolder
- C105: renamed from C108; footprint Capacitor_SMD:C_0603_1608Metric_Pad1.08x0.95mm_HandSolder -> Capacitor_SMD:C_0402_1005Metric_Pad0.74x0.62mm_HandSolder
- C106: renamed from C104; footprint Capacitor_SMD:C_0603_1608Metric_Pad1.08x0.95mm_HandSolder -> Capacitor_SMD:C_0402_1005Metric_Pad0.74x0.62mm_HandSolder
- C107: renamed from C109; footprint Capacitor_SMD:C_0603_1608Metric_Pad1.08x0.95mm_HandSolder -> Capacitor_SMD:C_0402_1005Metric_Pad0.74x0.62mm_HandSolder
- C108: renamed from C107; footprint Capacitor_SMD:C_0603_1608Metric_Pad1.08x0.95mm_HandSolder -> Capacitor_SMD:C_0402_1005Metric_Pad0.74x0.62mm_HandSolder
- C109: renamed from C110; footprint Capacitor_SMD:C_0603_1608Metric_Pad1.08x0.95mm_HandSolder -> Capacitor_SMD:C_0402_1005Metric_Pad0.74x0.62mm_HandSolder
- C110: renamed from C111; footprint Capacitor_SMD:C_0603_1608Metric_Pad1.08x0.95mm_HandSolder -> Capacitor_SMD:C_0402_1005Metric_Pad0.74x0.62mm_HandSolder
- C111: renamed from C112; footprint Capacitor_SMD:C_0603_1608Metric_Pad1.08x0.95mm_HandSolder -> Capacitor_SMD:C_0402_1005Metric_Pad0.74x0.62mm_HandSolder
- D101: renamed from D102; footprint LED_SMD:LED_0603_1608Metric_Pad1.05x0.95mm_HandSolder -> Resistor_SMD:R_0402_1005Metric_Pad0.72x0.64mm_HandSolder
- L101: footprint Inductor_SMD:L_0603_1608Metric_Pad1.05x0.95mm_HandSolder -> Capacitor_SMD:C_0402_1005Metric_Pad0.74x0.62mm_HandSolder
- R101: renamed from R102; footprint Resistor_SMD:R_0603_1608Metric_Pad0.98x0.95mm_HandSolder -> Resistor_SMD:R_0402_1005Metric_Pad0.72x0.64mm_HandSolder
- R102: renamed from R103; footprint Resistor_SMD:R_0603_1608Metric_Pad0.98x0.95mm_HandSolder -> Resistor_SMD:R_0402_1005Metric_Pad0.72x0.64mm_HandSolder
- U101: footprint Package_DFN_QFN:QFN-48-1EP_7x7mm_P0.5mm_EP5.6x5.6mm -> STM32:QFN-48-1EP_7x7mm_P0.5mm_EP5.6x5.6mm_AJ
- renumbered C103 to C102
Connections:
- net +3.3V: now also J101.2 (Pin_2)
- net GND: now also H101.1, H102.1, H103.1, H104.1, J101.1 (Pin_1)
- net CB_OUT3: now reaches U101.10 (PA2)
- net CB_OUT4: now reaches U101.11 (PA3)
- net CB_IN: now reaches U101.12 (PA4)
- net M_SCTR_LIDAR: now reaches U101.14 (PA6)
- net DEV_EN_LIDAR: now reaches U101.15 (PA7)
- net M_EN_LIDAR: now reaches U101.16 (PC4)
- net GPIO1: now reaches U101.2 (PC13)
- net GPIO1: now also J102.1 (Pin_1)
- net TX_LIDAR: now reaches U101.22 (PB10)
- net RX_LIDAR: now reaches U101.24 (PB11)
- net CHAT/SOURIS: now reaches U101.25 (PB12)
- net REV2: now reaches U101.26 (PB13)
- net REV1: now reaches U101.27 (PB14)
- net PHASE_B2: now reaches U101.29 (PC6)
- net GPIO2: now reaches U101.3 (PC14)
- net GPIO2: now also J102.2 (Pin_2)
- net FWD2: now reaches U101.30 (PA8)
- net FWD1: now reaches U101.31 (PA9)
- net PHASE_B1: now reaches U101.33 (PA11)
- net PHASE_A1: now reaches U101.34 (PA12)
- net SWDIO: now reaches U101.36 (PA13)
- net SWCLK: now reaches U101.37 (PA14)
- net TX_SWD: now reaches U101.39 (PC10)
- net GPIO3: now reaches U101.4 (PC15)
- net GPIO3: now also J102.3 (Pin_3)
- net RX_SWD: now reaches U101.40 (PC11)
- net SWO: now reaches U101.41 (PB3)
- net PHASE_A2: now reaches U101.43 (PB5)
- net INT1_ACCELERO: now reaches U101.44 (PB6)
- net SDA_ACCELERO: now reaches U101.45 (PB7)
- net SDA_ACCELERO: now also J101.3 (Pin_3)
- net SCL_ACCELERO: now reaches U101.46 (PB8)
- net SCL_ACCELERO: now also J101.4 (Pin_4)
- net CB_OUT2: now reaches U101.8 (PA0)
- net CB_OUT1: now reaches U101.9 (PA1)
- net VREF+ renamed VDDA
- no-connect marks 0 -> 9
Other:
- moved on the sheet: C106, C108

Commit message: commit AL08_1
Parts:
- removed J102: GPIO, Connector_PinSocket_2.54mm:PinSocket_1x03_P2.54mm_Vertical, symbol Connector:Screw_Terminal_01x03
- added D102: LED_USER1, Resistor_SMD:R_0402_1005Metric_Pad0.72x0.64mm_HandSolder, symbol Device:LED
- added D103: LED_USER2, Resistor_SMD:R_0402_1005Metric_Pad0.72x0.64mm_HandSolder, symbol Device:LED
- added D104: LED_USER3, Resistor_SMD:R_0402_1005Metric_Pad0.72x0.64mm_HandSolder, symbol Device:LED
- added R103: 1.5k, Resistor_SMD:R_0402_1005Metric_Pad0.72x0.64mm_HandSolder, symbol Device:R_Small
- added R104, R105, R106: 680, Resistor_SMD:R_0402_1005Metric_Pad0.72x0.64mm_HandSolder, symbol Device:R_Small
Connections:
- net GND: now also R103.2, R104.2, R105.2, R106.2
- net GPIO1: now also D102.2 (A)
- net GPIO2: now also D103.2 (A)
- net GPIO3: now also D104.2 (A)
- net SCL_ACCELERO: now also U101.38 (PA15); no longer U101.46 (PB8)
- new net: R103.1, U101.46 (PB8)
- new net: D104.1 (K), R106.1
- new net: D103.1 (K), R105.1
- new net: D102.1 (K), R104.1
- no-connect marks 9 -> 8

Commit message: commit du code et kicad modifié
Parts:
- removed C101, C104: 10p, Capacitor_SMD:C_0402_1005Metric_Pad0.74x0.62mm_HandSolder, symbol Device:C_Small
- removed C102: 4.7u, Capacitor_SMD:C_0603_1608Metric_Pad1.08x0.95mm_HandSolder, symbol Device:C_Small
- removed C103, C105, C107, C108, C109: 100n, Capacitor_SMD:C_0402_1005Metric_Pad0.74x0.62mm_HandSolder, symbol Device:C_Small
- removed C106, C111: 1u, Capacitor_SMD:C_0402_1005Metric_Pad0.74x0.62mm_HandSolder, symbol Device:C_Small
- removed C110: 10n, Capacitor_SMD:C_0402_1005Metric_Pad0.74x0.62mm_HandSolder, symbol Device:C_Small
- removed D101: LED_POWER, Resistor_SMD:R_0402_1005Metric_Pad0.72x0.64mm_HandSolder, symbol Device:LED
- removed D102: LED_USER1, Resistor_SMD:R_0402_1005Metric_Pad0.72x0.64mm_HandSolder, symbol Device:LED
- removed D103: LED_USER2, Resistor_SMD:R_0402_1005Metric_Pad0.72x0.64mm_HandSolder, symbol Device:LED
- removed D104: LED_USER3, Resistor_SMD:R_0402_1005Metric_Pad0.72x0.64mm_HandSolder, symbol Device:LED
- removed J101: ECRAN, Connector_PinSocket_2.54mm:PinSocket_1x04_P2.54mm_Vertical, symbol Connector:Screw_Terminal_01x04
- removed L101: l, Capacitor_SMD:C_0402_1005Metric_Pad0.74x0.62mm_HandSolder, symbol Device:L_Small
- removed R101, R104, R105, R106: 680, Resistor_SMD:R_0402_1005Metric_Pad0.72x0.64mm_HandSolder, symbol Device:R_Small
- removed R102: 20, Resistor_SMD:R_0402_1005Metric_Pad0.72x0.64mm_HandSolder, symbol Device:R_Small
- removed R103: 1.5k, Resistor_SMD:R_0402_1005Metric_Pad0.72x0.64mm_HandSolder, symbol Device:R_Small
- removed U101: STM32G431CBUx, STM32:QFN-48-1EP_7x7mm_P0.5mm_EP5.6x5.6mm_AJ, symbol MCU_ST_STM32G4:STM32G431CBUx
- removed Y101: 16MHz, Crystal:Crystal_SMD_3225-4Pin_3.2x2.5mm, symbol Device:Crystal_GND24_Small
Connections:
- no-connect marks 8 -> 0
Other:
- added sheet Actionneur (Actionneur.kicad_sch)
- added sheet STM32 (STM32.kicad_sch)
- sheet Alimentation ports: added 3.3V; removed none
- sheet SENSORS ports: added CB_IN, CB_OUT1, CB_OUT2, CB_OUT3, CB_OUT4, CHAT/SOURIS, DEV_EN_LIDAR, INT1_ACCELERO, MOTEUR1+, MOTEUR1-, MOTEUR2+, MOTEUR2-, M_EN_LIDAR, M_SCTR_LIDAR, PHASE_A1, PHASE_A2, PHASE_B1, PHASE_B2, RX_LIDAR, SCL, SDA, TX_LIDAR; removed none

Commit message: commit pour le schema
Other:
- sheet Actionneur ports: added BATT; removed none
- sheet Alimentation ports: added 5v, BATT; removed none
- sheet SENSORS ports: added 5v; removed none
- sheet STM32 ports: added 3.3V; removed none
- moved on the sheet: H101, H102, H103, H104

Commit message: commit pour le schema avec 2 CB
Parts:
- renumbered H101 to H1, H102 to H2, H103 to H3, H104 to H4
Other:
- sheet SENSORS ports: added none; removed CB_OUT3, CB_OUT4
- sheet STM32 ports: added none; removed CB_OUT3, CB_OUT4
Changed lines of the file:
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@@
-	)
-	(junction
-		(at 120.65 64.77)
-		(diameter 0)
-		(color 0 0 0 0)
 	)
 	(junction
@@
 	(wire
 		(pts
-			(xy 83.82 64.77) (xy 120.65 64.77)
-		)
-		(stroke
-			(width 0)
-			(type default)
-		)
-	)
-	(wire
-		(pts
 			(xy 88.9 35.56) (xy 57.15 35.56)
 		)
@@
 		(pts
 			(xy 148.59 147.32) (xy 97.79 147.32)
-		)
-		(stroke
-			(width 0)
-			(type default)
-		)
-	)
-	(wire
-		(pts
-			(xy 83.82 68.58) (xy 120.65 68.58)
 		)
 		(stroke
@@
 		(on_board yes)
 		(dnp no)
-		(property "Reference" "H104"
+		(property "Reference" "H4"
 			(at 264.414 88.138 0)
 			(effects
@@
 			(project "ESE_AL8"
 				(path "/c3d0eb52-cd9d-4e69-bcf7-3f0716f715c6"
-					(reference "H104")
+					(reference "H4")
 					(unit 1)
 				)
@@
 		(on_board yes)
 		(dnp no)
-		(property "Reference" "H103"
+		(property "Reference" "H3"
 			(at 259.334 88.138 0)
 			(effects
@@
 			(project "ESE_AL8"
 				(path "/c3d0eb52-cd9d-4e69-bcf7-3f0716f715c6"
-					(reference "H103")
+					(reference "H3")
 					(unit 1)
 				)
@@
 		(on_board yes)
 		(dnp no)
-		(property "Reference" "H101"
+		(property "Reference" "H1"
 			(at 249.174 88.138 0)
 			(effects
@@
 			(project ""
 				(path "/c3d0eb52-cd9d-4e69-bcf7-3f0716f715c6"
-					(reference "H101")
+					(reference "H1")
 					(unit 1)
 				)
@@
 		(dnp no)
 		(fields_autoplaced yes)
-		(property "Reference" "#PWR0114"
+		(property "Reference" "#PWR01"
 			(at 259.08 104.14 0)
 			(effects
@@
 			(project "ESE_AL8"
 				(path "/c3d0eb52-cd9d-4e69-bcf7-3f0716f715c6"
-					(reference "#PWR0114")
+					(reference "#PWR01")
 					(unit 1)
 				)
@@
 		(on_board yes)
 		(dnp no)
-		(property "Reference" "H102"
+		(property "Reference" "H2"
 			(at 254.254 88.138 0)
 			(effects
@@
 			(project "ESE_AL8"
 				(path "/c3d0eb52-cd9d-4e69-bcf7-3f0716f715c6"
-					(reference "H102")
+					(reference "H2")
 					(unit 1)
 				)
@@
 	(sheet
 		(at 120.65 49.53)
-		(size 46.99 91.44)
+		(size 46.99 87.376)
 		(fields_autoplaced yes)
 		(stroke
@@
 		)
 		(property "Sheetfile" "STM32.kicad_sch"
-			(at 120.65 141.5546 0)
+			(at 120.65 137.4906 0)
 			(effects
 				(font
@@
 		(pin "DEV_EN_LIDAR" input
 			(at 120.65 80.01 180)
-			(effects
-				(font
-					(size 1.27 1.27)
-				)
-				(justify left)
-			)
-		)
-		(pin "CB_OUT4" input
-			(at 120.65 68.58 180)
-			(effects
-				(font
-					(size 1.27 1.27)
-				)
-				(justify left)
-			)
-		)
-		(pin "CB_OUT3" input
-			(at 120.65 64.77 180)
 			(effects
 				(font
@@
 	)
 	(sheet
-		(at 215.9 21.59)
+		(at 233.934 48.768)
 		(size 48.26 30.48)
 		(fields_autoplaced yes)
@@
 		)
 		(property "Sheetname" "Schema architectural"
-			(at 215.9 20.8784 0)
+			(at 233.934 48.0564 0)
 			(effects
 				(font
@@
 		)
 		(property "Sheetfile" "schema_architectural.kicad_sch"
-			(at 215.9 52.6546 0)
+			(at 233.934 79.8326 0)
 			(effects
 				(font
@@
 			(effects
 				(font
-					(size 1.27 1.27)
-				)
-				(justify right)
-			)
-		)
-		(pin "CB_OUT4" input
-			(at 83.82 68.58 0)
-			(effects
-				(font
-					(size 1.27 1.27)
-				)
-				(justify right)
-			)
-		)
-		(pin "CB_OUT3" input
-			(at 83.82 64.77 0)
-			(effects
-				(font
