File: Schema_KICAD/ESE_AL8/ESE_AL8/ESE_AL8.kicad_sch (KiCad schematic)
At the start: 4 parts

Commit message: Commit last modif 23/10/24 11:29
Other:
- sheet Alimentation ports: added none; removed 3.3V
- sheet STM32 ports: added none; removed 3.3V
Changed lines of the file:
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@@
-	(wire
-		(pts
-			(xy 144.78 33.02) (xy 144.78 49.53)
-		)
-		(stroke
-			(width 0)
-			(type default)
-		)
-	)
 	(wire
 		(pts
@@
 		(pts
 			(xy 144.78 149.86) (xy 92.71 149.86)
-		)
-		(stroke
-			(width 0)
-			(type default)
-		)
-	)
-	(wire
-		(pts
-			(xy 127 33.02) (xy 144.78 33.02)
 		)
 		(stroke
@@
 			)
 		)
-		(pin "3.3V" input
-			(at 144.78 49.53 90)
-			(effects
-				(font
-					(size 1.27 1.27)
-				)
-				(justify right)
-			)
-		)
 		(pin "INT2_ACCELERO" input
 			(at 120.65 110.49 180)
@@
 			)
 		)
-		(pin "3.3V" input
-			(at 127 33.02 0)
-			(effects
-				(font
-					(size 1.27 1.27)
-				)
-				(justify right)
-			)
-		)
