File: Schema_KICAD/ESE_AL8/ESE_AL8/schema_architectural.kicad_sch (KiCad schematic)
At the start: 0 parts

Commit message: schema
Other:
- note added: "2 LED"
- note added: "2*Capteur Bordeur"
- note added: "2*Driver"
- note added: "2*Moteur"
- note added: "3.3V"
- note added: "5V"
- note added: "Accelerometre"
- note added: "Batterie JST 7.2V"
- note added: "GPIOs"
- note added: "I2C"
- note added: "Interrupteur Chat/Souris"
- note added: "LIDAR 5V"
- note added: "MCU"
- note added: "Quartz"
- note added: "SPI"
- note added: "SWD/JIAG"
- note added: "USART"

Commit message: LE 25 /09/2024 10:31
Other:
- note added: "4*Capteur Bordeur"
- note added: "Pour les encodeurs"
- note removed: "2*Capteur Bordeur"
Changed lines of the file:
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@@
 	)
 	(rectangle
-		(start 147.32 73.66)
-		(end 147.32 87.63)
+		(start 141.986 73.66)
+		(end 141.986 87.63)
+		(stroke
+			(width 0)
+			(type default)
+		)
+		(fill
+			(type none)
+		)
+	)
+	(rectangle
+		(start 204.47 76.2)
+		(end 204.47 76.962)
 		(stroke
 			(width 0)
@@
 	)
 	(rectangle
-		(start 156.21 81.28)
-		(end 182.88 81.28)
-		(stroke
-			(width 0)
-			(type default)
-		)
-		(fill
-			(type none)
-		)
-	)
-	(rectangle
-		(start 201.93 48.26)
-		(end 201.93 80.01)
-		(stroke
-			(width 0)
-			(type default)
-		)
-		(fill
-			(type none)
-		)
-	)
-	(rectangle
 		(start 160.02 101.6)
 		(end 160.02 113.03)
@@
 	)
 	(rectangle
-		(start 125.73 43.18)
-		(end 125.73 48.26)
-		(stroke
-			(width 0)
-			(type default)
-		)
-		(fill
-			(type none)
-		)
-	)
-	(rectangle
-		(start 193.04 80.01)
-		(end 193.04 80.01)
+		(start 223.52 81.026)
+		(end 223.52 90.17)
+		(stroke
+			(width 0)
+			(type default)
+		)
+		(fill
+			(type none)
+		)
+	)
+	(rectangle
+		(start 162.306 89.154)
+		(end 181.61 89.154)
 		(stroke
 			(width 0)
@@
 	)
 	(rectangle
-		(start 154.94 53.34)
-		(end 154.94 87.63)
-		(stroke
-			(width 0)
-			(type default)
-		)
-		(fill
-			(type none)
-		)
-	)
-	(rectangle
-		(start 182.88 53.34)
-		(end 182.88 58.42)
+		(start 181.61 94.996)
+		(end 181.61 95.25)
+		(stroke
+			(width 0)
+			(type default)
+		)
+		(fill
+			(type none)
+		)
+	)
+	(rectangle
+		(start 149.86 53.34)
+		(end 149.86 87.63)
+		(stroke
+			(width 0)
+			(type default)
+		)
+		(fill
+			(type none)
+		)
+	)
+	(rectangle
+		(start 129.286 89.916)
+		(end 140.716 89.916)
+		(stroke
+			(width 0)
+			(type default)
+		)
+		(fill
+			(type none)
+		)
+	)
+	(rectangle
+		(start 162.306 93.98)
+		(end 201.422 93.98)
 		(stroke
 			(width 0)
@@
 	)
 	(rectangle
-		(start 182.88 73.66)
-		(end 182.88 81.28)
-		(stroke
-			(width 0)
-			(type default)
-		)
-		(fill
-			(type none)
-		)
-	)
-	(rectangle
 		(start 93.98 63.754)
 		(end 119.38 80.264)
@@
 	)
 	(rectangle
-		(start 165.1 58.42)
-		(end 199.39 73.66)
-		(stroke
-			(width 0)
-			(type default)
-		)
-		(fill
-			(type none)
-		)
-	)
-	(rectangle
-		(start 181.61 90.17)
-		(end 200.66 99.06)
+		(start 151.13 61.214)
+		(end 185.42 76.454)
+		(stroke
+			(width 0)
+			(type default)
+		)
+		(fill
+			(type none)
+		)
+	)
+	(rectangle
+		(start 181.61 81.28)
+		(end 181.61 86.868)
+		(stroke
+			(width 0)
+			(type default)
+		)
+		(fill
+			(type none)
+		)
+	)
+	(rectangle
+		(start 129.286 71.12)
+		(end 129.286 89.916)
+		(stroke
+			(width 0)
+			(type default)
+		)
+		(fill
+			(type none)
+		)
+	)
+	(rectangle
+		(start 195.072 76.962)
+		(end 214.122 85.852)
+		(stroke
+			(width 0)
+			(type default)
+		)
+		(fill
+			(type none)
+		)
+	)
+	(rectangle
+		(start 181.61 86.614)
+		(end 181.61 89.154)
 		(stroke
 			(width 0)
@@
 	)
 	(rectangle
+		(start 181.61 81.28)
+		(end 182.118 81.28)
+		(stroke
+			(width 0)
+			(type default)
+		)
+		(fill
+			(type none)
+		)
+	)
+	(rectangle
 		(start 86.614 120.396)
 		(end 102.87 130.556)
@@
 	)
 	(rectangle
-		(start 193.04 80.01)
-		(end 201.93 80.01)
-		(stroke
-			(width 0)
-			(type default)
-		)
-		(fill
-			(type none)
-		)
-	)
-	(rectangle
-		(start 125.73 48.26)
-		(end 201.93 48.26)
-		(stroke
-			(width 0)
-			(type default)
-		)
-		(fill
-			(type none)
-		)
-	)
-	(rectangle
 		(start 119.38 24.13)
 		(end 119.38 29.21)
@@
 	(rectangle
 		(start 121.92 53.34)
-		(end 182.88 53.34)
+		(end 149.86 53.34)
 		(stroke
 			(width 0)
@@
 	)
 	(rectangle
-		(start 193.04 80.01)
-		(end 193.04 90.17)
-		(stroke
-			(width 0)
-			(type default)
-		)
-		(fill
-			(type none)
-		)
-	)
-	(rectangle
 		(start 204.47 43.18)
-		(end 204.47 82.55)
-		(stroke
-			(width 0)
-			(type default)
-		)
-		(fill
-			(type none)
-		)
-	)
-	(rectangle
-		(start 138.43 61.976)
-		(end 153.67 73.66)
+		(end 204.47 76.2)
+		(stroke
+			(width 0)
+			(type default)
+		)
+		(fill
+			(type none)
+		)
+	)
+	(rectangle
+		(start 133.096 61.976)
+		(end 148.336 73.66)
 		(stroke
 			(width 0)
@@
 	)
 	(rectangle
+		(start 119.38 71.12)
+		(end 129.286 71.12)
+		(stroke
+			(width 0)
+			(type default)
+		)
+		(fill
+			(type none)
+		)
+	)
+	(rectangle
 		(start 194.31 100.33)
 		(end 194.31 111.76)
@@
 	)
 	(rectangle
+		(start 156.21 76.454)
+		(end 156.21 81.534)
+		(stroke
+			(width 0)
+			(type default)
+		)
+		(fill
+			(type none)
+		)
+	)
+	(rectangle
 		(start 156.21 81.28)
 		(end 156.21 87.63)
@@
 	)
 	(rectangle
+		(start 182.118 81.28)
+		(end 195.072 81.28)
+		(stroke
+			(width 0)
+			(type default)
+		)
+		(fill
+			(type none)
+		)
+	)
+	(rectangle
 		(start 204.47 107.95)
 		(end 245.11 107.95)
@@
 	)
 	(rectangle
-		(start 195.58 82.55)
-		(end 204.47 82.55)
-		(stroke
-			(width 0)
-			(type default)
-		)
-		(fill
-			(type none)
-		)
-	)
-	(rectangle
 		(start 119.38 25.4)
 		(end 119.38 25.4)
@@
 	)
 	(rectangle
-		(start 162.56 95.25)
-		(end 181.61 95.25)
-		(stroke
-			(width 0)
-			(type default)
-		)
-		(fill
-			(type none)
-		)
-	)
-	(rectangle
 		(start 140.716 87.376)
 		(end 162.306 102.616)
@@
 	)
 	(rectangle
-		(start 195.58 82.55)
-		(end 195.58 90.17)
+		(start 214.122 81.026)
+		(end 223.52 81.026)
 		(stroke
 			(width 0)
@@
 	(text "2 LED"
 		(exclude_from_sim no)
-		(at 146.304 68.58 0)
+		(at 140.97 68.58 0)
 		(effects
 			(font
@@
 	(text "Interrupteur\n\nChat/Souris"
 		(exclude_from_sim no)
-		(at 182.88 65.786 0)
-		(effects
-			(font
-				(size 1.778 1.778)
+		(at 168.91 68.58 0)
+		(effects
+			(font
+				(size 1.778 1.778)
+			)
+		)
+	)
+	(text "Pour les encodeurs"
+		(exclude_from_sim no)
+		(at 202.184 92.71 0)
+		(effects
+			(font
+				(size 1.27 1.27)
 			)
 		)
@@
 	(text "2*Driver"
 		(exclude_from_sim no)
-		(at 192.024 94.996 0)
-		(effects
-			(font
-				(size 1.778 1.778)
-			)
-		)
-	)
-	(text "2*Capteur Bordeur"
+		(at 205.486 81.788 0)
+		(effects
+			(font
+				(size 1.778 1.778)
+			)
+		)
+	)
+	(text "Pour les encodeurs"
+		(exclude_from_sim no)
+		(at 231.14 68.326 90)
+		(effects
+			(font
+				(size 1.27 1.27)
+			)
+		)
+	)
+	(text "4*Capteur Bordeur"
 		(exclude_from_sim no)
 		(at 199.39 118.11 0)

Commit message: commit du code et kicad modifié
Other:
- note added: "GPIOs(si possible)"
- note removed: "GPIOs"
Changed lines of the file:
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@@
 	)
 	(rectangle
-		(start 66.04 102.87)
-		(end 82.296 113.03)
+		(start 60.706 105.156)
+		(end 85.852 113.03)
 		(stroke
 			(width 0)
@@
 		)
 	)
-	(text "GPIOs\n"
-		(exclude_from_sim no)
-		(at 73.406 108.204 0)
-		(effects
-			(font
+	(text "GPIOs(si possible)\n\n"
+		(exclude_from_sim no)
+		(at 73.152 111.252 0)
+		(effects
+			(font

Commit message: commit pour le schema avec 2 CB
Other:
- note added: "2*Capteur bordure"
- note removed: "4*Capteur Bordeur"
Changed lines of the file:
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@@
 		)
 	)
-	(text "4*Capteur Bordeur"
+	(text "2*Capteur bordure"
 		(exclude_from_sim no)
 		(at 199.39 118.11 0)
