File: Schema_KICAD/ESE_AL8/ESE_AL8/alimentation.kicad_sch (KiCad schematic)
At the start: 19 parts, among them IC301 MP1475SGJ-P, J301 Batterie, U301 BUxxSD5

Commit message: commit pour 18/09
Parts:
- renumbered C306 to C302, C302 to C303, C303 to C304, C304 to C305, C305 to C306, R302 to R301, R303 to R302, R301 to R303, R306 to R305, R305 to R306
Changed lines of the file:
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@@
 		(dnp no)
 		(fields_autoplaced yes)
-		(property "Reference" "#PWR0307"
+		(property "Reference" "#PWR0310"
 			(at 226.06 83.82 0)
 			(effects
@@
 			(project "ESE_AL8"
 				(path "/c3d0eb52-cd9d-4e69-bcf7-3f0716f715c6/f403419b-15e7-44f7-a652-fb424ff9de0d"
-					(reference "#PWR0307")
+					(reference "#PWR0310")
 					(unit 1)
 				)
@@
 		(on_board yes)
 		(dnp no)
-		(property "Reference" "C305"
+		(property "Reference" "C306"
 			(at 216.662 45.212 0)
 			(effects
@@
 			(project "ESE_AL8"
 				(path "/c3d0eb52-cd9d-4e69-bcf7-3f0716f715c6/f403419b-15e7-44f7-a652-fb424ff9de0d"
-					(reference "C305")
+					(reference "C306")
 					(unit 1)
 				)
@@
 		(dnp no)
 		(fields_autoplaced yes)
-		(property "Reference" "#PWR0309"
+		(property "Reference" "#PWR0308"
 			(at 217.17 132.08 0)
 			(effects
@@
 			(project "ESE_AL8"
 				(path "/c3d0eb52-cd9d-4e69-bcf7-3f0716f715c6/f403419b-15e7-44f7-a652-fb424ff9de0d"
-					(reference "#PWR0309")
+					(reference "#PWR0308")
 					(unit 1)
 				)
@@
 		(on_board yes)
 		(dnp no)
-		(property "Reference" "C302"
+		(property "Reference" "C303"
 			(at 126.492 38.989 0)
 			(effects
@@
 			(project "ESE_AL8"
 				(path "/c3d0eb52-cd9d-4e69-bcf7-3f0716f715c6/f403419b-15e7-44f7-a652-fb424ff9de0d"
-					(reference "C302")
+					(reference "C303")
 					(unit 1)
 				)
@@
 		(dnp no)
 		(fields_autoplaced yes)
-		(property "Reference" "#PWR0306"
+		(property "Reference" "#PWR0302"
 			(at 119.126 85.344 0)
 			(effects
@@
 			(project "ESE_AL8"
 				(path "/c3d0eb52-cd9d-4e69-bcf7-3f0716f715c6/f403419b-15e7-44f7-a652-fb424ff9de0d"
-					(reference "#PWR0306")
+					(reference "#PWR0302")
 					(unit 1)
 				)
@@
 		(on_board yes)
 		(dnp no)
-		(property "Reference" "#PWR0304"
+		(property "Reference" "#PWR0305"
 			(at 207.645 55.88 0)
 			(effects
@@
 			(project "ESE_AL8"
 				(path "/c3d0eb52-cd9d-4e69-bcf7-3f0716f715c6/f403419b-15e7-44f7-a652-fb424ff9de0d"
-					(reference "#PWR0304")
+					(reference "#PWR0305")
 					(unit 1)
 				)
@@
 		(on_board yes)
 		(dnp no)
-		(property "Reference" "#PWR0308"
+		(property "Reference" "#PWR0306"
 			(at 210.185 97.155 0)
 			(effects
@@
 			(project "ESE_AL8"
 				(path "/c3d0eb52-cd9d-4e69-bcf7-3f0716f715c6/f403419b-15e7-44f7-a652-fb424ff9de0d"
-					(reference "#PWR0308")
+					(reference "#PWR0306")
 					(unit 1)
 				)
@@
 		(on_board yes)
 		(dnp no)
-		(property "Reference" "R301"
+		(property "Reference" "R303"
 			(at 189.738 31.75 90)
 			(effects
@@
 			(project "ESE_AL8"
 				(path "/c3d0eb52-cd9d-4e69-bcf7-3f0716f715c6/f403419b-15e7-44f7-a652-fb424ff9de0d"
-					(reference "R301")
+					(reference "R303")
 					(unit 1)
 				)
@@
 		(on_board yes)
 		(dnp no)
-		(property "Reference" "C303"
+		(property "Reference" "C304"
 			(at 185.166 39.624 0)
 			(effects
@@
 			(project "ESE_AL8"
 				(path "/c3d0eb52-cd9d-4e69-bcf7-3f0716f715c6/f403419b-15e7-44f7-a652-fb424ff9de0d"
-					(reference "C303")
+					(reference "C304")
 					(unit 1)
 				)
@@
 		(on_board yes)
 		(dnp no)
-		(property "Reference" "R305"
+		(property "Reference" "R306"
 			(at 220.98 87.63 90)
 			(effects
@@
 			(project "ESE_AL8"
 				(path "/c3d0eb52-cd9d-4e69-bcf7-3f0716f715c6/f403419b-15e7-44f7-a652-fb424ff9de0d"
-					(reference "R305")
+					(reference "R306")
 					(unit 1)
 				)
@@
 		(on_board yes)
 		(dnp no)
-		(property "Reference" "C304"
+		(property "Reference" "C305"
 			(at 206.375 44.45 0)
 			(effects
@@
 			(project "ESE_AL8"
 				(path "/c3d0eb52-cd9d-4e69-bcf7-3f0716f715c6/f403419b-15e7-44f7-a652-fb424ff9de0d"
-					(reference "C304")
+					(reference "C305")
 					(unit 1)
 				)
@@
 		(dnp no)
 		(fields_autoplaced yes)
-		(property "Reference" "#PWR0305"
+		(property "Reference" "#PWR0304"
 			(at 149.86 80.01 0)
 			(effects
@@
 			(project "ESE_AL8"
 				(path "/c3d0eb52-cd9d-4e69-bcf7-3f0716f715c6/f403419b-15e7-44f7-a652-fb424ff9de0d"
-					(reference "#PWR0305")
+					(reference "#PWR0304")
 					(unit 1)
 				)
@@
 		(on_board yes)
 		(dnp no)
-		(property "Reference" "R303"
+		(property "Reference" "R302"
 			(at 110.49 76.962 0)
 			(effects
@@
 			(project "ESE_AL8"
 				(path "/c3d0eb52-cd9d-4e69-bcf7-3f0716f715c6/f403419b-15e7-44f7-a652-fb424ff9de0d"
-					(reference "R303")
+					(reference "R302")
 					(unit 1)
 				)
@@
 		(on_board yes)
 		(dnp no)
-		(property "Reference" "R302"
+		(property "Reference" "R301"
 			(at 105.664 39.497 0)
 			(effects
@@
 			(project "ESE_AL8"
 				(path "/c3d0eb52-cd9d-4e69-bcf7-3f0716f715c6/f403419b-15e7-44f7-a652-fb424ff9de0d"
-					(reference "R302")
+					(reference "R301")
 					(unit 1)
 				)
@@
 		(dnp no)
 		(fields_autoplaced yes)
-		(property "Reference" "#PWR0313"
+		(property "Reference" "#PWR0311"
 			(at 233.68 142.24 0)
 			(effects
@@
 			(project "ESE_AL8"
 				(path "/c3d0eb52-cd9d-4e69-bcf7-3f0716f715c6/f403419b-15e7-44f7-a652-fb424ff9de0d"
-					(reference "#PWR0313")
+					(reference "#PWR0311")
 					(unit 1)
 				)
@@
 		(dnp no)
 		(fields_autoplaced yes)
-		(property "Reference" "#PWR0311"
+		(property "Reference" "#PWR0309"
 			(at 217.17 139.7 0)
 			(effects
@@
 			(project "ESE_AL8"
 				(path "/c3d0eb52-cd9d-4e69-bcf7-3f0716f715c6/f403419b-15e7-44f7-a652-fb424ff9de0d"
-					(reference "#PWR0311")
+					(reference "#PWR0309")
 					(unit 1)
 				)
@@
 		(on_board yes)
 		(dnp no)
-		(property "Reference" "R306"
+		(property "Reference" "R305"
 			(at 212.09 88.265 0)
 			(effects
@@
 			(project "ESE_AL8"
 				(path "/c3d0eb52-cd9d-4e69-bcf7-3f0716f715c6/f403419b-15e7-44f7-a652-fb424ff9de0d"
-					(reference "R306")
+					(reference "R305")
 					(unit 1)
 				)
@@
 		(dnp no)
 		(fields_autoplaced yes)
-		(property "Reference" "#PWR0302"
+		(property "Reference" "#PWR0307"
 			(at 217.17 46.355 0)
 			(effects
@@
 			(project "ESE_AL8"
 				(path "/c3d0eb52-cd9d-4e69-bcf7-3f0716f715c6/f403419b-15e7-44f7-a652-fb424ff9de0d"
-					(reference "#PWR0302")
+					(reference "#PWR0307")
 					(unit 1)
 				)
@@
 		(on_board yes)
 		(dnp no)
-		(property "Reference" "C306"
+		(property "Reference" "C302"
 			(at 121.158 75.946 0)
 			(effects
@@
 			(project "ESE_AL8"
 				(path "/c3d0eb52-cd9d-4e69-bcf7-3f0716f715c6/f403419b-15e7-44f7-a652-fb424ff9de0d"
-					(reference "C306")
+					(reference "C302")
 					(unit 1)
 				)
@@
 		(dnp no)
 		(fields_autoplaced yes)
-		(property "Reference" "#PWR0310"
+		(property "Reference" "#PWR0313"
 			(at 250.063 132.08 0)
 			(effects
@@
 			(project "ESE_AL8"
 				(path "/c3d0eb52-cd9d-4e69-bcf7-3f0716f715c6/f403419b-15e7-44f7-a652-fb424ff9de0d"
-					(reference "#PWR0310")
-					(unit 1)
-				)
+					(reference "#PWR0313")
+					(unit 1)
+				)

Commit message: LE 25 /09/2024 10:31
Parts:
- added SW301: ON/OFF, STM32:SWITCH TOGGLE SPDT 1A 30V, symbol Switch:SW_SPDT_321
- C302, C303, C304, C307, C308, C309: footprint Capacitor_SMD:C_0603_1608Metric_Pad1.08x0.95mm_HandSolder -> Capacitor_SMD:C_0402_1005Metric_Pad0.74x0.62mm_HandSolder
- L301: footprint Inductor_SMD:L_0603_1608Metric_Pad1.05x0.95mm_HandSolder -> Capacitor_SMD:C_0402_1005Metric_Pad0.74x0.62mm_HandSolder
- R301, R302, R303, R304, R305, R306: footprint Resistor_SMD:R_0603_1608Metric_Pad0.98x0.95mm_HandSolder -> Resistor_SMD:R_0402_1005Metric_Pad0.72x0.64mm_HandSolder
Connections:
- net GND: now also SW301.3 (A)
- net VIN: now also SW301.2 (B); no longer J301.1 (Pin_1)
- new net +7.2V: J301.1 (Pin_1), SW301.1 (C)
Other:
- moved on the sheet: J301

Commit message: commit du code et kicad modifié
Parts:
- removed C301: 22u, Capacitor_SMD:C_0603_1608Metric_Pad1.08x0.95mm_HandSolder, symbol Device:C_Small
- removed C302, C303: 0.1u, Capacitor_SMD:C_0402_1005Metric_Pad0.74x0.62mm_HandSolder, symbol Device:C_Small
- removed R301, R302: 100K, Resistor_SMD:R_0402_1005Metric_Pad0.72x0.64mm_HandSolder, symbol Device:R_Small
- added C21: 22u, Capacitor_SMD:C_0603_1608Metric_Pad1.08x0.95mm_HandSolder, symbol Device:C_Small
- added C22, C23: 0.1u, Capacitor_SMD:C_0402_1005Metric_Pad0.74x0.62mm_HandSolder, symbol Device:C_Small
- added D1: LED_POWER, Resistor_SMD:R_0402_1005Metric_Pad0.72x0.64mm_HandSolder, symbol Device:LED
- added R1: 680, Resistor_SMD:R_0402_1005Metric_Pad0.72x0.64mm_HandSolder, symbol Device:R_Small
- added R7, R8: 100K, Resistor_SMD:R_0402_1005Metric_Pad0.72x0.64mm_HandSolder, symbol Device:R_Small
- C308, C309: value 0.47u -> 1u
- SW301: footprint STM32:SWITCH TOGGLE SPDT 1A 30V -> Connector_JST:JST_EH_B3B-EH-A_1x03_P2.50mm_Vertical
Connections:
- net +3.3V: now also D1.2 (A)
- net GND: now also C21.2, C22.2, C23.2, R1.2
- net BST: no longer names the net of IC301.5 (BST), R303.1
- net EN/SYNC: no longer names the net of IC301.6 (EN/SYNC)
- net EN/SYNC: now also R7.2
- net FB: no longer names the net of IC301.8 (FB), R304.1
- net PG: no longer names the net of IC301.1 (PG)
- net PG: now also R8.2
- net SW: no longer names the net of C304.2, IC301.3 (SW), L301.1
- net VCC: no longer names the net of IC301.7 (VCC)
- net VCC: now also C22.1, R8.1
- net VIN renamed +BATT
- net +BATT: now also C21.1, C23.1, R7.1
- new net: D1.1 (K), R1.1
Other:
- note added: "LED ALIM"
- moved on the sheet: C304, C305, C306, C307, IC301, L301, R303, R304, R305, R306

Commit message: commit pour le schema
Changed lines of the file:
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@@
 	(wire
 		(pts
-			(xy 216.535 54.61) (xy 219.075 54.61)
+			(xy 216.535 54.61) (xy 223.52 54.61)
 		)
 		(stroke
@@
 		)
 	)
+	(hierarchical_label "5v"
+		(shape input)
+		(at 219.71 54.61 90)
+		(fields_autoplaced yes)
+		(effects
+			(font
+				(size 1.27 1.27)
+			)
+			(justify left)
+		)
+	)
+	(hierarchical_label "BATT"
+		(shape input)
+		(at 115.57 46.99 90)
+		(fields_autoplaced yes)
+		(effects
+			(font
+				(size 1.27 1.27)
+			)
+			(justify left)
+		)
+	)
 	(hierarchical_label "3.3V"
 		(shape input)
@@
 	(symbol
 		(lib_id "power:+5V")
-		(at 219.075 54.61 0)
+		(at 223.52 54.61 0)
 		(unit 1)
 		(exclude_from_sim no)
@@
 		(fields_autoplaced yes)
 		(property "Reference" "#PWR0308"
-			(at 219.075 58.42 0)
+			(at 223.52 58.42 0)
 			(effects
 				(font
@@
 		)
 		(property "Value" "+5V"
-			(at 219.075 49.53 0)
+			(at 223.52 49.53 0)
 			(effects
 				(font
@@
 		)
 		(property "Footprint" ""
-			(at 219.075 54.61 0)
+			(at 223.52 54.61 0)
 			(effects
 				(font
@@
 		)
 		(property "Datasheet" ""
-			(at 219.075 54.61 0)
-			(effects
-				(font
-					(size 1.27 1.27)
-				)
-				(hide yes)
-			)
-		)
-		(property "Description" ""
-			(at 219.075 54.61 0)
-			(effects
-				(font
+			(at 223.52 54.61 0)
+			(effects
+				(font
+					(size 1.27 1.27)
+				)
+				(hide yes)
+			)
+		)
+		(property "Description" ""
+			(at 223.52 54.61 0)
+			(effects
+				(font

Commit message: commit pour le schema avec 2 CB
Parts:
- J6: renamed from J301; footprint Connector_JST:JST_EH_B2B-EH-A_1x02_P2.50mm_Vertical -> Connector_JST:JST_XH_S2B-XH-A_1x02_P2.50mm_Horizontal
- SW2: renamed from SW301; footprint Connector_JST:JST_EH_B3B-EH-A_1x03_P2.50mm_Vertical -> Connector_JST:JST_XH_S3B-XH-A_1x03_P2.50mm_Horizontal
- renumbered C308 to C10, C309 to C11, C21 to C3, C23 to C4, C22 to C5, C304 to C6, C307 to C7, C305 to C8, C306 to C9, IC301 to IC1, L301 to L1, R1 to R3, R7 to R4, R8 to R5, R303 to R6, R304 to R7, R305 to R8, R306 to R9, U301 to U2
Connections:
- net +7.2V: now also SW2.3 (A); no longer SW2.1 (C)
- net GND: now also SW2.1 (C); no longer SW2.3 (A)
- net sw: now reaches C6.2, IC1.3 (SW), L1.1
- net en/sync: now reaches IC1.6 (EN/SYNC), R4.2
- net vcc: now reaches C5.1, IC1.7 (VCC), R5.1
- net pg: now reaches IC1.1 (PG), R5.2
- net led_power: now reaches D1.1 (K), R3.1
- net fb: now reaches IC1.8 (FB), R7.1
- net bst: now reaches IC1.5 (BST), R6.1
Other:
- moved on the sheet: C3, C4, C6, C7, C8, C9, L1, R4, R6, R7, R8, R9

Commit message: commit pour le placement des composants 12h
Parts:
- C3, C8, C9: footprint Capacitor_SMD:C_0603_1608Metric_Pad1.08x0.95mm_HandSolder -> Capacitor_SMD:C_0805_2012Metric_Pad1.18x1.45mm_HandSolder
Connections:
- net GND: no longer SW2.1 (C)
- no-connect marks 1 -> 2
Other:
- moved on the sheet: R5
Changed lines of the file:
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@@
 		(at 241.3 132.08)
 	)
-	(wire
-		(pts
-			(xy 120.65 66.04) (xy 120.65 68.58)
+	(no_connect
+		(at 58.42 43.18)
+	)
+	(wire
+		(pts
+			(xy 124.46 66.04) (xy 124.46 68.58)
 		)
 		(stroke
@@
 	(wire
 		(pts
-			(xy 120.65 59.69) (xy 133.35 59.69)
+			(xy 124.46 59.69) (xy 133.35 59.69)
 		)
 		(stroke
@@
 	(wire
 		(pts
-			(xy 120.65 68.58) (xy 143.51 68.58)
+			(xy 124.46 68.58) (xy 143.51 68.58)
 		)
 		(stroke
@@
 	(wire
 		(pts
-			(xy 120.65 60.96) (xy 120.65 59.69)
+			(xy 124.46 60.96) (xy 124.46 59.69)
 		)
 		(stroke
@@
 	(symbol
 		(lib_id "Device:R_Small")
-		(at 120.65 63.5 0)
+		(at 124.46 63.5 0)
 		(unit 1)
 		(exclude_from_sim no)
@@
 		(dnp no)
 		(property "Reference" "R5"
-			(at 121.92 62.992 0)
+			(at 125.73 62.992 0)
 			(effects
 				(font
@@
 		)
 		(property "Value" "100K"
-			(at 122.428 64.77 0)
+			(at 126.238 64.77 0)
 			(effects
 				(font
@@
 		)
 		(property "Footprint" "Resistor_SMD:R_0402_1005Metric_Pad0.72x0.64mm_HandSolder"
-			(at 120.65 63.5 0)
+			(at 124.46 63.5 0)
 			(effects
 				(font
@@
 		)
 		(property "Datasheet" "~"
-			(at 120.65 63.5 0)
+			(at 124.46 63.5 0)
 			(effects
 				(font
@@
 		)
 		(property "Description" ""
-			(at 120.65 63.5 0)
+			(at 124.46 63.5 0)
 			(effects
 				(font
@@
 			)
 		)
-		(property "Footprint" "Capacitor_SMD:C_0603_1608Metric_Pad1.08x0.95mm_HandSolder"
+		(property "Footprint" "Capacitor_SMD:C_0805_2012Metric_Pad1.18x1.45mm_HandSolder"
 			(at 216.535 59.055 0)
 			(effects
@@
 			)
 		)
-		(property "Footprint" "Capacitor_SMD:C_0603_1608Metric_Pad1.08x0.95mm_HandSolder"
+		(property "Footprint" "Capacitor_SMD:C_0805_2012Metric_Pad1.18x1.45mm_HandSolder"
 			(at 107.95 54.61 0)
 			(effects
@@
 	)
 	(symbol
-		(lib_id "power:GND")
-		(at 58.42 43.18 0)
-		(unit 1)
-		(exclude_from_sim no)
-		(in_bom yes)
-		(on_board yes)
-		(dnp no)
-		(property "Reference" "#PWR020"
-			(at 58.42 49.53 0)
-			(effects
-				(font
-					(size 1.27 1.27)
-				)
-				(hide yes)
-			)
-		)
-		(property "Value" "GND"
-			(at 55.118 44.704 0)
-			(effects
-				(font
-					(size 1.27 1.27)
-				)
-			)
-		)
-		(property "Footprint" ""
-			(at 58.42 43.18 0)
-			(effects
-				(font
-					(size 1.27 1.27)
-				)
-				(hide yes)
-			)
-		)
-		(property "Datasheet" ""
-			(at 58.42 43.18 0)
-			(effects
-				(font
-					(size 1.27 1.27)
-				)
-				(hide yes)
-			)
-		)
-		(property "Description" ""
-			(at 58.42 43.18 0)
-			(effects
-				(font
-					(size 1.27 1.27)
-				)
-				(hide yes)
-			)
-		)
-		(pin "1"
-		)
-		(instances
-			(project "ESE_AL8"
-				(path "/c3d0eb52-cd9d-4e69-bcf7-3f0716f715c6/f403419b-15e7-44f7-a652-fb424ff9de0d"
-					(reference "#PWR020")
-					(unit 1)
-				)
-			)
-		)
-	)
-	(symbol
 		(lib_id "Device:C_Small")
 		(at 205.74 58.42 0)
@@
 			)
 		)
-		(property "Footprint" "Capacitor_SMD:C_0603_1608Metric_Pad1.08x0.95mm_HandSolder"
+		(property "Footprint" "Capacitor_SMD:C_0805_2012Metric_Pad1.18x1.45mm_HandSolder"
 			(at 205.74 58.42 0)
 			(effects
