File: Schema_KICAD/ESE_AL8/ESE_AL8/alimentation.kicad_sch (KiCad schematic)
At the start: 22 parts, among them IC1 MP1475SGJ-P, J6 Batterie, SW2 ON/OFF, U2 BUxxSD5

Commit message: Commit midif pcb 2020
Parts:
- added D5, D6: LED_POWER, LED_SMD:LED_0603_1608Metric, symbol Device:LED
- added R14, R15: 680, Resistor_SMD:R_0402_1005Metric, symbol Device:R_Small
- R6, R7, R8, R9: footprint Resistor_SMD:R_0402_1005Metric -> Resistor_SMD:R_0603_1608Metric
Connections:
- net +5V: now also D5.2 (A)
- net +BATT: now also D6.2 (A)
- net GND: now also R14.2, R15.2
- new net led_power5: D5.1 (K), R14.1
- new net led_powerBATT: D6.1 (K), R15.1

Commit message: le bon ioc
Parts:
- R14: value 680 -> 2.5
- R15: value 680 -> 4.2
- R3: value 680 -> 1k
Other:
- moved on the sheet: C10, C11, C3, C4, C5, C6, C7, C8, C9, D1, D5, D6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
