File: Schema_KICAD/ESE_AL8/ESE_AL8/Actionneur.kicad_sch (KiCad schematic)
At the start: 15 parts, among them J1 ECRAN, U2 ZXBM5210-SP, U3 ZXBM5210-SP

Commit message: commit pour le schema
Changed lines of the file:
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@@
+		)
+	)
+	(hierarchical_label "BATT"
+		(shape input)
+		(at 64.77 55.88 90)
+		(fields_autoplaced yes)
+		(effects
+			(font
+				(size 1.27 1.27)
+			)
+			(justify left)
 		)
 	)

Commit message: commit pour le schema avec 2 CB
Parts:
- C29: renamed from C25; footprint Capacitor_SMD:C_0603_1608Metric_Pad1.08x0.95mm_HandSolder -> Capacitor_SMD:C_0402_1005Metric_Pad0.74x0.62mm_HandSolder
- J8: renamed from J1; footprint Connector_JST:JST_EH_B4B-EH-A_1x04_P2.50mm_Vertical -> Connector_JST:JST_XH_S4B-XH-A_1x04_P2.50mm_Horizontal
- TP4: renamed from TP5; footprint (none) -> TestPoint:TestPoint_Pad_D1.0mm
- TP5: renamed from TP6; footprint (none) -> TestPoint:TestPoint_Pad_D1.0mm
- TP6: renamed from TP3; footprint (none) -> TestPoint:TestPoint_Pad_D1.0mm
- TP7: renamed from TP4; footprint (none) -> TestPoint:TestPoint_Pad_D1.0mm
- renumbered C17 to C24, C18 to C25, C19 to C26, C20 to C27, C24 to C28, C16 to C30, C14 to C31, U2 to U4, U3 to U5

Commit message: commit pour le placement des composants 12h
Parts:
- C28: footprint Capacitor_SMD:C_0402_1005Metric_Pad0.74x0.62mm_HandSolder -> Capacitor_SMD:C_0603_1608Metric_Pad1.08x0.95mm_HandSolder
Changed lines of the file:
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@@
 			)
 		)
-		(property "Footprint" "Capacitor_SMD:C_0402_1005Metric_Pad0.74x0.62mm_HandSolder"
+		(property "Footprint" "Capacitor_SMD:C_0603_1608Metric_Pad1.08x0.95mm_HandSolder"
 			(at 113.03 142.24 0)
 			(effects

Commit message: commit pour le schema aprés routage
Parts:
- C24, C25, C26, C27, C29, C31: footprint Capacitor_SMD:C_0402_1005Metric_Pad0.74x0.62mm_HandSolder -> Capacitor_SMD:C_0402_1005Metric
- C28, C30: footprint Capacitor_SMD:C_0603_1608Metric_Pad1.08x0.95mm_HandSolder -> Capacitor_SMD:C_0603_1608Metric
- U4, U5: footprint Package_SO:Diodes_SO-8EP -> STM32:Diodes_SO-8EP
Changed lines of the file:
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@@
 			)
 		)
-		(property "Footprint" "Capacitor_SMD:C_0402_1005Metric_Pad0.74x0.62mm_HandSolder"
+		(property "Footprint" "Capacitor_SMD:C_0402_1005Metric"
 			(at 120.65 142.24 0)
 			(effects
@@
 			)
 		)
-		(property "Footprint" "Capacitor_SMD:C_0603_1608Metric_Pad1.08x0.95mm_HandSolder"
+		(property "Footprint" "Capacitor_SMD:C_0603_1608Metric"
 			(at 125.73 64.77 0)
 			(effects
@@
 			)
 		)
-		(property "Footprint" "Capacitor_SMD:C_0402_1005Metric_Pad0.74x0.62mm_HandSolder"
+		(property "Footprint" "Capacitor_SMD:C_0402_1005Metric"
 			(at 97.79 67.31 0)
 			(effects
@@
 			)
 		)
-		(property "Footprint" "Capacitor_SMD:C_0402_1005Metric_Pad0.74x0.62mm_HandSolder"
+		(property "Footprint" "Capacitor_SMD:C_0402_1005Metric"
 			(at 130.81 64.77 0)
 			(effects
@@
 			)
 		)
-		(property "Footprint" "Capacitor_SMD:C_0402_1005Metric_Pad0.74x0.62mm_HandSolder"
+		(property "Footprint" "Capacitor_SMD:C_0402_1005Metric"
 			(at 87.63 144.78 0)
 			(effects
@@
 			)
 		)
-		(property "Footprint" "Capacitor_SMD:C_0603_1608Metric_Pad1.08x0.95mm_HandSolder"
+		(property "Footprint" "Capacitor_SMD:C_0603_1608Metric"
 			(at 113.03 142.24 0)
 			(effects
@@
 			)
 		)
-		(property "Footprint" "Package_SO:Diodes_SO-8EP"
+		(property "Footprint" "STM32:Diodes_SO-8EP"
 			(at 74.93 156.21 0)
 			(effects
@@
 			)
 		)
-		(property "Footprint" "Capacitor_SMD:C_0402_1005Metric_Pad0.74x0.62mm_HandSolder"
+		(property "Footprint" "Capacitor_SMD:C_0402_1005Metric"
 			(at 96.52 82.55 0)
 			(effects
@@
 			)
 		)
-		(property "Footprint" "Capacitor_SMD:C_0402_1005Metric_Pad0.74x0.62mm_HandSolder"
+		(property "Footprint" "Capacitor_SMD:C_0402_1005Metric"
 			(at 86.36 154.94 0)
 			(effects
@@
 			)
 		)
-		(property "Footprint" "Package_SO:Diodes_SO-8EP"
+		(property "Footprint" "STM32:Diodes_SO-8EP"
 			(at 83.82 73.66 0)
 			(effects
