File: Schema_KICAD/ESE_AL8/ESE_AL8/Actionneur.kicad_sch (KiCad schematic)
At the start: 15 parts, among them J8 ECRAN, U4 ZXBM5210-SP, U5 ZXBM5210-SP

Commit message: new version
Other:
- moved on the sheet: J8

Commit message: commit
Other:
- moved on the sheet: J8
