File: Schema_KICAD/ESE_AL8/ESE_AL8/ESE_AL8.kicad_pcb (KiCad board)
At the start: 4 copper layers, 60 x 60 mm, 70 parts, among them IC301 MP1475SGJ-P, J101 ECRAN, J102 GPIO, J201 JTAG/SWD, J202 Moteur1, J203 Moteur2, J204 LIDAR, J205 CB1, J206 CB2, J207 CB3, J208 CB4, J301 Batterie, SW201 SW_c/s, SW301 ON/OFF, U101 STM32G431CBUx, U201 ZXBM5210-SP, U202 ZXBM5210-SP, U203 ADXL343, U301 BUxxSD5, Y101 16MHz

Commit message: commit 3
Routing:
- net VIN: track 149.0 -> 0.00 mm, vias 2 -> 1
- net +5V: track 62.1 -> 0.00 mm, vias 1 -> 0
- net +3.3V: track 50.9 -> 0.00 mm, vias 8 -> 0
- net SCL_ACCELERO: track 49.6 -> 0.00 mm
- net CB_IN: track 46.0 -> 0.00 mm
- net SWO: track 44.3 -> 0.00 mm
- net PHASE_A2: track 43.7 -> 0.00 mm, vias 1 -> 0
- net PHASE_B1: track 41.2 -> 0.00 mm, vias 1 -> 0
- net PHASE_A1: track 38.9 -> 0.00 mm, vias 1 -> 0
- net NRST: track 37.5 -> 0.00 mm, vias 2 -> 0
- net SDA_ACCELERO: track 36.3 -> 0.00 mm
- net FWD1: track 33.9 -> 0.00 mm
- net RX_LIDAR: track 33.0 -> 0.00 mm
- net SWDIO: track 31.2 -> 0.00 mm
- net GPIO1: track 31.0 -> 0.00 mm
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- added copper zone on In2.Cu, net VIN
- removed copper zone on In2.Cu, net +3.3V

Commit message: commit du code et kicad modifié
Parts:
- removed C101, C104: 10p, Capacitor_SMD:C_0402_1005Metric_Pad0.74x0.62mm_HandSolder
- removed C102: 4.7u, Capacitor_SMD:C_0603_1608Metric_Pad1.08x0.95mm_HandSolder
- removed C103, C105, C107, C108, C109, C205, C206, C207, C208: 100n, Capacitor_SMD:C_0402_1005Metric_Pad0.74x0.62mm_HandSolder
- removed C106, C111, C201, C202, C209, C210: 1u, Capacitor_SMD:C_0402_1005Metric_Pad0.74x0.62mm_HandSolder
- removed C110: 10n, Capacitor_SMD:C_0402_1005Metric_Pad0.74x0.62mm_HandSolder
- removed C203, C204: 10u, Capacitor_SMD:C_0603_1608Metric_Pad1.08x0.95mm_HandSolder
- removed C308, C309: 0.47u, Capacitor_SMD:C_0402_1005Metric_Pad0.74x0.62mm_HandSolder
- removed D101: LED_POWER, Resistor_SMD:R_0402_1005Metric_Pad0.72x0.64mm_HandSolder
- removed H101, H102, H103, H104: MountingHole_Pad, MountingHole:MountingHole_3.2mm_M3_Pad_Via
- removed J101: ECRAN, Connector_PinSocket_2.54mm:PinSocket_1x04_P2.54mm_Vertical
- removed J102: GPIO, Connector_PinSocket_2.54mm:PinSocket_1x03_P2.54mm_Vertical
- removed J201: JTAG/SWD, Connector_PinHeader_1.27mm:PinHeader_2x07_P1.27mm_Vertical_SMD
- removed J202: Moteur1, Connector_JST:JST_EH_B6B-EH-A_1x06_P2.50mm_Vertical
- removed J203: Moteur2, Connector_JST:JST_EH_B6B-EH-A_1x06_P2.50mm_Vertical
- removed J204: LIDAR, Connector_JST:JST_EH_B7B-EH-A_1x07_P2.50mm_Vertical
- removed J205: CB1, Connector_JST:JST_EH_B4B-EH-A_1x04_P2.50mm_Vertical
- removed J206: CB2, Connector_JST:JST_EH_B4B-EH-A_1x04_P2.50mm_Vertical
- removed J207: CB3, Connector_JST:JST_EH_B4B-EH-A_1x04_P2.50mm_Vertical
- removed J208: CB4, Connector_JST:JST_EH_B4B-EH-A_1x04_P2.50mm_Vertical
- removed J301: Batterie, Connector_JST:JST_EH_B2B-EH-A_1x02_P2.50mm_Vertical
- removed JP201: TestRX, Jumper:SolderJumper-2_P1.3mm_Open_TrianglePad1.0x1.5mm
- removed JP202: TestTX, Jumper:SolderJumper-2_P1.3mm_Open_TrianglePad1.0x1.5mm
- removed L101: l, Capacitor_SMD:C_0402_1005Metric_Pad0.74x0.62mm_HandSolder
- removed R101: 680, Resistor_SMD:R_0402_1005Metric_Pad0.72x0.64mm_HandSolder
- removed R102: 20, Resistor_SMD:R_0402_1005Metric_Pad0.72x0.64mm_HandSolder
- removed R201, R202: 2.2k, Resistor_SMD:R_0402_1005Metric_Pad0.72x0.64mm_HandSolder
- removed SW201: SW_c/s, Button_Switch_SMD:SW_Push_1P1T_NO_6x6mm_H9.5mm
- removed SW301: ON/OFF, STM32:SWITCH TOGGLE SPDT 1A 30V
- removed TP201: TestPoint, TestPoint:TestPoint_Pad_D1.0mm
- removed U101: STM32G431CBUx, STM32:QFN-48-1EP_7x7mm_P0.5mm_EP5.6x5.6mm_AJ
- removed U201, U202: ZXBM5210-SP, Package_SO:Diodes_SO-8EP
- removed U203: ADXL343, Package_LGA:LGA-14_3x5mm_P0.8mm_LayoutBorder1x6y
- removed U301: BUxxSD5, Package_TO_SOT_SMD:SOT-23-5_HandSoldering
- removed Y101: 16MHz, Crystal:Crystal_SMD_3225-4Pin_3.2x2.5mm
- moved C305 31.9 mm to (142.7, 103.2), turned to 90 degrees
- moved C306 29.7 mm to (144.3, 103.3), turned to 90 degrees
- moved C303 28.6 mm to (140.7, 95.0), turned to -90 degrees
- moved C301 27.9 mm to (142.0, 95.6), turned to -90 degrees
- moved L301 23.6 mm to (149.0, 103.1), turned to -90 degrees
- moved R301 22.7 mm to (141.5, 92.0), turned to 90 degrees
- moved R302 19.9 mm to (145.3, 90.4), turned to -90 degrees
- moved IC301 16.8 mm to (147.2, 94.9), turned to 0 degrees
- moved C304 16.1 mm to (152.5, 100.1), turned to -90 degrees
- moved R303 14.3 mm to (150.3, 99.5), turned to 0 degrees
- moved R305 10.6 mm to (150.4, 91.0), turned to 180 degrees
- moved C302 10.1 mm to (151.6, 95.2)
- moved R304 9.82 mm to (150.3, 92.3), turned to 0 degrees
- moved C307 2.27 mm to (154.3, 93.0), turned to 0 degrees
- moved R306 2.13 mm to (154.4, 94.3), turned to 0 degrees
Routing:
- net VCC: track 0.00 -> 15.5 mm, vias 0 -> 2
- net EN/SYNC: track 0.00 -> 15.4 mm, vias 0 -> 2
- net +5V: track 0.00 -> 8.50 mm, vias 0 -> 2
- net VIN: track 0.00 -> 7.23 mm, vias 1 -> 0
- net SW: track 0.00 -> 6.82 mm, vias 0 -> 2
- net Net-(C307-Pad1): track 0.00 -> 5.70 mm
- net BST: track 0.00 -> 4.74 mm, vias 0 -> 2
- net PG: track 0.00 -> 2.73 mm
- net FB: track 0.00 -> 1.96 mm
- net Net-(C304-Pad1): track 0.00 -> 1.66 mm
- added copper zone on In2.Cu, net +5V
- added copper zone on In2.Cu, net SW
- removed copper zone on B.Cu, net GND
- removed copper zone on In1.Cu, net GND
Other:
- board outline removed

Commit message: commit pour le schema avec 2 CB
Parts:
- removed C301, C305, C306: 22u, Capacitor_SMD:C_0603_1608Metric_Pad1.08x0.95mm_HandSolder
- removed C302, C303, C304: 0.1u, Capacitor_SMD:C_0402_1005Metric_Pad0.74x0.62mm_HandSolder
- removed C307: 15p, Capacitor_SMD:C_0402_1005Metric_Pad0.74x0.62mm_HandSolder
- removed IC301: MP1475SGJ-P, Package_TO_SOT_SMD:TSOT-23-8_HandSoldering
- removed L301: 4.7u, Capacitor_SMD:C_0402_1005Metric_Pad0.74x0.62mm_HandSolder
- removed R301, R302: 100K, Resistor_SMD:R_0402_1005Metric_Pad0.72x0.64mm_HandSolder
- removed R303: 20, Resistor_SMD:R_0402_1005Metric_Pad0.72x0.64mm_HandSolder
- removed R304: 16k, Resistor_SMD:R_0402_1005Metric_Pad0.72x0.64mm_HandSolder
- removed R305: 7.68k, Resistor_SMD:R_0402_1005Metric_Pad0.72x0.64mm_HandSolder
- removed R306: 40.2k, Resistor_SMD:R_0402_1005Metric_Pad0.72x0.64mm_HandSolder
- added C12: 10p, Capacitor_SMD:C_0402_1005Metric_Pad0.74x0.62mm_HandSolder, F.Cu at (140.8, 97.2)
- added C13: 4.7u, Capacitor_SMD:C_0402_1005Metric_Pad0.74x0.62mm_HandSolder, F.Cu at (147.1, 94.1)
- added C14: 100n, Capacitor_SMD:C_0402_1005Metric_Pad0.74x0.62mm_HandSolder, F.Cu at (146.1, 95.8)
- added C15: 1u, Capacitor_SMD:C_0402_1005Metric_Pad0.74x0.62mm_HandSolder, F.Cu at (151.6, 105.5)
- added C16: 10p, Capacitor_SMD:C_0402_1005Metric_Pad0.74x0.62mm_HandSolder, F.Cu at (139.4, 101.7)
- added C17: 100n, Capacitor_SMD:C_0402_1005Metric_Pad0.74x0.62mm_HandSolder, F.Cu at (148.1, 94.1)
- added C18: 100n, Capacitor_SMD:C_0402_1005Metric_Pad0.74x0.62mm_HandSolder, F.Cu at (150.6, 105.5)
- added C19: 100n, Capacitor_SMD:C_0402_1005Metric_Pad0.74x0.62mm_HandSolder, F.Cu at (155.1, 104.0)
- added C21: 100n, Capacitor_SMD:C_0402_1005Metric_Pad0.74x0.62mm_HandSolder, F.Cu at (156.8, 97.0)
- added C22: 10n, Capacitor_SMD:C_0402_1005Metric_Pad0.74x0.62mm_HandSolder, F.Cu at (154.7, 106.0)
- added C23: 1u, Capacitor_SMD:C_0402_1005Metric_Pad0.74x0.62mm_HandSolder, F.Cu at (152.6, 105.5)
- added D2: LED_USER1, Resistor_SMD:R_0402_1005Metric_Pad0.72x0.64mm_HandSolder, F.Cu at (140.7, 93.2)
- added D3: LED_USER2, Resistor_SMD:R_0402_1005Metric_Pad0.72x0.64mm_HandSolder, F.Cu at (140.7, 94.2)
- added D4: LED_USER3, Resistor_SMD:R_0402_1005Metric_Pad0.72x0.64mm_HandSolder, F.Cu at (140.7, 95.2)
- added H1: MountingHole_Pad, MountingHole:MountingHole_3.2mm_M3_Pad_Via, F.Cu at (134.0, 69.9)
- added H2: MountingHole_Pad, MountingHole:MountingHole_3.2mm_M3_Pad_Via, F.Cu at (180.0, 70.0)
- added H3: MountingHole_Pad, MountingHole:MountingHole_3.2mm_M3_Pad_Via, F.Cu at (180.0, 119.0)
- added H4: MountingHole_Pad, MountingHole:MountingHole_3.2mm_M3_Pad_Via, F.Cu at (134.0, 119.0)
- added L2: l, Capacitor_SMD:C_0402_1005Metric_Pad0.74x0.62mm_HandSolder, F.Cu at (154.7, 105.0)
- added R10: 20, Resistor_SMD:R_0402_1005Metric_Pad0.72x0.64mm_HandSolder, F.Cu at (141.8, 101.7)
- added R11: 680, Resistor_SMD:R_0402_1005Metric_Pad0.72x0.64mm_HandSolder, F.Cu at (138.4, 93.2)
- added R12: 680, Resistor_SMD:R_0402_1005Metric_Pad0.72x0.64mm_HandSolder, F.Cu at (138.4, 94.2)
- added R13: 680, Resistor_SMD:R_0402_1005Metric_Pad0.72x0.64mm_HandSolder, F.Cu at (138.4, 95.2)
- added U3: STM32G431CBUx, STM32:QFN-48-1EP_7x7mm_P0.5mm_EP5.6x5.6mm_AJ, F.Cu at (151.4, 99.4)
- added Y1: 16MHz, Crystal:Crystal_SMD_3225-4Pin_3.2x2.5mm, F.Cu at (140.8, 99.5)
Routing:
- net VCC: track 15.5 -> 0.00 mm, vias 2 -> 0
- net EN/SYNC: track 15.4 -> 0.00 mm, vias 2 -> 0
- net +5V: track 8.50 -> 0.00 mm, vias 2 -> 0
- net VIN: track 7.23 -> 0.00 mm
- net SW: track 6.82 -> 0.00 mm, vias 2 -> 0
- net Net-(C307-Pad1): track 5.70 -> 0.00 mm
- net BST: track 4.74 -> 0.00 mm, vias 2 -> 0
- net PG: track 2.73 -> 0.00 mm
- net FB: track 1.96 -> 0.00 mm
- net Net-(C304-Pad1): track 1.66 -> 0.00 mm
- added copper zone on B.Cu, net GND
- added copper zone on In1.Cu, net GND
- removed copper zone on In2.Cu, net +5V
- removed copper zone on In2.Cu, net SW
- removed copper zone on In2.Cu, net VIN
Other:
- board outline added: 54 x 57 mm

Commit message: commit pour le placement des composants 12h
Parts:
- added C1: 1u, Capacitor_SMD:C_0402_1005Metric_Pad0.74x0.62mm_HandSolder, F.Cu at (60.2, 83.9)
- added C10: 1u, Capacitor_SMD:C_0402_1005Metric_Pad0.74x0.62mm_HandSolder, F.Cu at (59.8, 110.2)
- added C11: 1u, Capacitor_SMD:C_0402_1005Metric_Pad0.74x0.62mm_HandSolder, F.Cu at (65.7, 110.2)
- added C2: 100n, Capacitor_SMD:C_0402_1005Metric_Pad0.74x0.62mm_HandSolder, F.Cu at (60.2, 85.9)
- added C20: 100n, Capacitor_SMD:C_0402_1005Metric_Pad0.74x0.62mm_HandSolder, F.Cu at (148.2, 73.7)
- added C24: 100n, Capacitor_SMD:C_0402_1005Metric_Pad0.74x0.62mm_HandSolder, F.Cu at (66.8, 73.3)
- added C25: 100n, Capacitor_SMD:C_0402_1005Metric_Pad0.74x0.62mm_HandSolder, F.Cu at (66.8, 75.3)
- added C26: 100n, Capacitor_SMD:C_0402_1005Metric_Pad0.74x0.62mm_HandSolder, F.Cu at (66.8, 77.2)
- added C27: 100n, Capacitor_SMD:C_0402_1005Metric_Pad0.74x0.62mm_HandSolder, F.Cu at (66.8, 79.2)
- added C28: 10u, Capacitor_SMD:C_0603_1608Metric_Pad1.08x0.95mm_HandSolder, F.Cu at (66.8, 81.2)
- added C29: 1u, Capacitor_SMD:C_0402_1005Metric_Pad0.74x0.62mm_HandSolder, F.Cu at (66.8, 83.2)
- added C3: 22u, Capacitor_SMD:C_0805_2012Metric_Pad1.18x1.45mm_HandSolder, F.Cu at (161.4, 85.1)
- added C30: 10u, Capacitor_SMD:C_0603_1608Metric_Pad1.08x0.95mm_HandSolder, F.Cu at (81.7, 73.6)
- added C31: 1u, Capacitor_SMD:C_0402_1005Metric_Pad0.74x0.62mm_HandSolder, F.Cu at (66.8, 85.1)
- added C4: 0.1u, Capacitor_SMD:C_0402_1005Metric_Pad0.74x0.62mm_HandSolder, F.Cu at (160.7, 86.6)
- added C5: 0.1u, Capacitor_SMD:C_0402_1005Metric_Pad0.74x0.62mm_HandSolder, F.Cu at (162.0, 76.1)
- added C6: 0.1u, Capacitor_SMD:C_0402_1005Metric_Pad0.74x0.62mm_HandSolder, F.Cu at (165.6, 76.9)
- added C7: 15p, Capacitor_SMD:C_0402_1005Metric_Pad0.74x0.62mm_HandSolder, F.Cu at (159.4, 73.7)
- added C8: 22u, Capacitor_SMD:C_0805_2012Metric_Pad1.18x1.45mm_HandSolder, F.Cu at (166.7, 83.3)
- added C9: 22u, Capacitor_SMD:C_0805_2012Metric_Pad1.18x1.45mm_HandSolder, F.Cu at (166.7, 81.3)
- added D1: LED_POWER, Resistor_SMD:R_0402_1005Metric_Pad0.72x0.64mm_HandSolder, F.Cu at (66.8, 89.1)
- added IC1: MP1475SGJ-P, Package_TO_SOT_SMD:TSOT-23-8_HandSoldering, F.Cu at (161.5, 80.3)
- added J1: CB1, Connector_JST:JST_XH_S4B-XH-A_1x04_P2.50mm_Horizontal, F.Cu at (132.5, 90.9)
- added J2: CB2, Connector_JST:JST_XH_S4B-XH-A_1x04_P2.50mm_Horizontal, F.Cu at (132.5, 104.5)
- added J3: LIDAR, Connector_JST:JST_XH_S8B-XH-A_1x08_P2.50mm_Horizontal, F.Cu at (154.3, 120.2)
- added J4: Moteur1, Connector_JST:JST_XH_S6B-XH-A_1x06_P2.50mm_Horizontal, F.Cu at (181.5, 90.8)
- added J5: Moteur2, Connector_JST:JST_XH_S6B-XH-A_1x06_P2.50mm_Horizontal, F.Cu at (181.4, 110.5)
- added J6: Batterie, Connector_JST:JST_XH_S2B-XH-A_1x02_P2.50mm_Horizontal, F.Cu at (160.5, 68.5)
- added J7: Conn_ST_STDC14, Connector_PinHeader_1.27mm:PinHeader_2x07_P1.27mm_Vertical_SMD, F.Cu at (142.7, 71.0)
- added J8: ECRAN, Connector_JST:JST_XH_S4B-XH-A_1x04_P2.50mm_Horizontal, F.Cu at (132.5, 76.7)
- added L1: 4.7u, Capacitor_SMD:C_0402_1005Metric_Pad0.74x0.62mm_HandSolder, F.Cu at (168.9, 77.9)
- added R1: 1k, Resistor_SMD:R_0402_1005Metric_Pad0.72x0.64mm_HandSolder, F.Cu at (60.3, 80.0)
- added R2: 1k, Resistor_SMD:R_0402_1005Metric_Pad0.72x0.64mm_HandSolder, F.Cu at (60.3, 81.9)
- added R3: 680, Resistor_SMD:R_0402_1005Metric_Pad0.72x0.64mm_HandSolder, F.Cu at (63.6, 91.3)
- added R4: 100K, Resistor_SMD:R_0402_1005Metric_Pad0.72x0.64mm_HandSolder, F.Cu at (158.5, 83.5)
- added R5: 100K, Resistor_SMD:R_0402_1005Metric_Pad0.72x0.64mm_HandSolder, F.Cu at (158.5, 82.4)
- added R6: 20, Resistor_SMD:R_0402_1005Metric_Pad0.72x0.64mm_HandSolder, F.Cu at (163.8, 78.6)
- added R7: 16k, Resistor_SMD:R_0402_1005Metric_Pad0.72x0.64mm_HandSolder, F.Cu at (158.9, 77.9)
- added R8: 7.68k, Resistor_SMD:R_0402_1005Metric_Pad0.72x0.64mm_HandSolder, F.Cu at (157.9, 77.9)
- added R9: 40.2k, Resistor_SMD:R_0402_1005Metric_Pad0.72x0.64mm_HandSolder, F.Cu at (160.5, 73.8)
- added SW1: SW_c/s, Button_Switch_SMD:SW_Push_1P1T_NO_6x6mm_H9.5mm, F.Cu at (145.9, 119.5)
- added SW2: ON/OFF, Connector_JST:JST_XH_S3B-XH-A_1x03_P2.50mm_Horizontal, F.Cu at (171.9, 68.4)
- added TP1: TestPoint, TestPoint:TestPoint_Pad_D1.0mm, F.Cu at (60.2, 88.4)
- added TP2: TestPoint, TestPoint:TestPoint_Pad_D1.0mm, F.Cu at (60.2, 91.5)
- added TP3: TestPoint, TestPoint:TestPoint_Pad_D1.0mm, F.Cu at (60.2, 94.5)
- added TP4: TestPoint, TestPoint:TestPoint_Pad_D1.0mm, F.Cu at (78.0, 73.8)
- added TP5: TestPoint, TestPoint:TestPoint_Pad_D1.0mm, F.Cu at (78.0, 76.9)
- added TP6: TestPoint, TestPoint:TestPoint_Pad_D1.0mm, F.Cu at (78.0, 80.0)
- added TP7: TestPoint, TestPoint:TestPoint_Pad_D1.0mm, F.Cu at (78.0, 83.0)
- added U1: ADXL343, Package_LGA:LGA-14_3x5mm_P0.8mm_LayoutBorder1x6y, F.Cu at (148.2, 89.4)
- added U2: BUxxSD5, Package_TO_SOT_SMD:SOT-23-5_HandSoldering, F.Cu at (62.7, 110.9)
- added U4: ZXBM5210-SP, Package_SO:Diodes_SO-8EP, F.Cu at (173.6, 106.3)
- added U5: ZXBM5210-SP, Package_SO:Diodes_SO-8EP, F.Cu at (173.8, 87.3)
- moved C12 9.68 mm to (147.2, 104.4)
- moved C16 9.68 mm to (145.9, 108.9)
- moved R10 9.68 mm to (148.2, 108.9)
- moved Y1 9.68 mm to (147.2, 106.7)
- moved C14 8.70 mm to (151.0, 103.0)
- moved C19 8.70 mm to (160.1, 111.2)
- moved C22 8.70 mm to (159.6, 113.2)
- moved D2 8.70 mm to (145.7, 100.4)
- moved D3 8.70 mm to (145.7, 101.4)
- moved D4 8.70 mm to (145.7, 102.4)
- moved L2 8.70 mm to (159.6, 112.2)
- moved R11 8.70 mm to (143.4, 100.4)
- moved R12 8.70 mm to (143.4, 101.4)
- moved R13 8.70 mm to (143.4, 102.4)
- moved U3 8.70 mm to (156.4, 106.5)
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Connections:
- net GPIO1 renamed LD1
- net GPIO2 renamed LD2
- net GPIO3 renamed LD3
Routing:
- net /Actionneur/MOTEUR1+: track 0.00 -> 10.1 mm
- net /Actionneur/MOTEUR1-: track 0.00 -> 8.62 mm
- net +7.2V: track 0.00 -> 6.47 mm
- net /SENSORS/M_SCTR_LIDAR: track 0.00 -> 6.32 mm
- net /SENSORS/DEV_EN_LIDAR: track 0.00 -> 5.79 mm
- net /SENSORS/M_EN_LIDAR: track 0.00 -> 5.65 mm
- net +BATT: track 0.00 -> 3.73 mm
- net (no net): vias 0 -> 4

Commit message: commit pour le schema aprés routage
Parts:
- added C201: 100n, Capacitor_SMD:C_0402_1005Metric, F.Cu at (138.5, 117.0)
- added G***: LOGO, STM32:logo, B.Cu at (146.4, 108.5)
- C1, C10, C11, C12, C13, C14, C15, C16, C17, C18, C19, C2, C20, C21, C22, C23, C24, C25, C26, C27, C29, C31, C4, C5, C6, C7: footprint Capacitor_SMD:C_0402_1005Metric_Pad0.74x0.62mm_HandSolder -> Capacitor_SMD:C_0402_1005Metric
- C28, C30: footprint Capacitor_SMD:C_0603_1608Metric_Pad1.08x0.95mm_HandSolder -> Capacitor_SMD:C_0603_1608Metric
- C3, C8, C9: footprint Capacitor_SMD:C_0805_2012Metric_Pad1.18x1.45mm_HandSolder -> Capacitor_SMD:C_0805_2012Metric
- D1, D2, D3, D4: footprint Resistor_SMD:R_0402_1005Metric_Pad0.72x0.64mm_HandSolder -> LED_SMD:LED_0603_1608Metric
- IC1: footprint Package_TO_SOT_SMD:TSOT-23-8_HandSoldering -> Package_TO_SOT_SMD:TSOT-23-8
- L1: footprint Capacitor_SMD:C_0402_1005Metric_Pad0.74x0.62mm_HandSolder -> STM32:IND_052047_WRE
- R1, R10, R11, R12, R13, R2, R3, R4, R5, R6, R7, R8, R9: footprint Resistor_SMD:R_0402_1005Metric_Pad0.72x0.64mm_HandSolder -> Resistor_SMD:R_0402_1005Metric
- SW1: footprint Button_Switch_SMD:SW_Push_1P1T_NO_6x6mm_H9.5mm -> STM32:SW_Push_1P1T_NO_6x6mm_H9.5mm
- U2: footprint Package_TO_SOT_SMD:SOT-23-5_HandSoldering -> Package_TO_SOT_SMD:SOT-23-5
- U4, U5: footprint Package_SO:Diodes_SO-8EP -> STM32:Diodes_SO-8EP
- moved C25 113.9 mm to (177.1, 103.8), turned to 90 degrees
- moved C24 113.9 mm to (174.2, 111.2), turned to -90 degrees
- moved C27 110.6 mm to (177.3, 84.8), turned to 90 degrees
- moved C26 108.7 mm to (174.5, 92.1), turned to -90 degrees
- moved C28 108.6 mm to (173.7, 100.5), turned to 90 degrees
- moved C10 108.3 mm to (167.0, 94.9), turned to 90 degrees
- moved C29 107.1 mm to (172.4, 101.1), turned to 90 degrees
- moved C31 105.8 mm to (172.6, 82.1), turned to -90 degrees
- moved U2 102.7 mm to (164.1, 94.4), turned to 180 degrees
- moved TP5 97.4 mm to (169.7, 109.8)
- moved C11 96.7 mm to (161.1, 94.7), turned to 90 degrees
- moved TP4 96.6 mm to (170.0, 103.5)
- moved R3 96.1 mm to (158.3, 75.3)
- moved TP7 94.1 mm to (171.7, 91.9)
- moved C30 92.5 mm to (173.9, 81.5), turned to -90 degrees
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Routing:
- net /Actionneur/SDA: track 0.00 -> 46.6 mm
- net /Actionneur/SCL: track 0.00 -> 46.1 mm
- net NRST: track 0.00 -> 41.2 mm, vias 0 -> 2
- net RX_SWD: track 0.00 -> 40.4 mm
- net /SENSORS/PHASE_B1: track 0.00 -> 39.9 mm, vias 0 -> 1
- net /SENSORS/CB_IN: track 0.00 -> 38.6 mm
- net TX_SWD: track 0.00 -> 36.0 mm
- net SWDIO: track 0.00 -> 34.8 mm
- net SWCLK: track 0.00 -> 34.3 mm
- net SWO: track 0.00 -> 34.0 mm, vias 0 -> 2
- net /SENSORS/PHASE_A2: track 0.00 -> 31.8 mm, vias 0 -> 1
- net /SENSORS/CB_OUT1: track 0.00 -> 31.5 mm
- net /Actionneur/FWD1: track 0.00 -> 30.3 mm
- net /SENSORS/PHASE_A1: track 0.00 -> 29.6 mm, vias 0 -> 1
- net +3.3V: track 0.00 -> 27.0 mm, vias 0 -> 9
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- added copper zone on In2.Cu, net +3.3V
- added copper zone on In2.Cu, net +5V
- added copper zone on In2.Cu, net +BATT
