File: Schema_KICAD/ESE_AL8/ESE_AL8/ESE_AL8.kicad_pcb (KiCad board)
At the start: 4 copper layers, 54 x 57 mm, 79 parts, among them IC1 MP1475SGJ-P, J1 CB1, J2 CB2, J3 LIDAR, J4 Moteur1, J5 Moteur2, J6 Batterie, J7 Conn_ST_STDC14, J8 ECRAN, SW1 SW_c/s, SW2 ON/OFF, U1 ADXL343, U2 BUxxSD5, U3 STM32G431CBUx, U4 ZXBM5210-SP, U5 ZXBM5210-SP, Y1 16MHz

Commit message: Commit midif pcb 2020
Parts:
- added D5: LED_POWER, LED_SMD:LED_0603_1608Metric, F.Cu at (165.8, 98.5)
- added D6: LED_POWER, LED_SMD:LED_0603_1608Metric, F.Cu at (168.5, 75.6)
- added R14: 680, Resistor_SMD:R_0402_1005Metric, F.Cu at (163.1, 98.6)
- added R15: 680, Resistor_SMD:R_0402_1005Metric, F.Cu at (171.1, 75.5)
- added R16: 1k, Resistor_SMD:R_0402_1005Metric, F.Cu at (138.9, 114.9)
- added R17: 1k, Resistor_SMD:R_0402_1005Metric, F.Cu at (140.8, 114.9)
- R6, R7, R8, R9: footprint Resistor_SMD:R_0402_1005Metric -> Resistor_SMD:R_0603_1608Metric
- moved C7 2.06 mm to (167.8, 90.0)
- moved R8 1.40 mm to (167.8, 87.3)
- moved R9 1.38 mm to (166.2, 89.4)
- moved R6 0.55 mm to (160.2, 85.5)
- moved C6 0.50 mm to (159.2, 86.8)
- moved C21 0.36 mm to (161.4, 103.5)
- moved R7 0.16 mm to (166.1, 86.2)
Connections:
- SW1 pad 1: /SENSORS/CHAT/SOURIS -> Net-(R16-Pad2)
Routing:
- net Net-(R16-Pad2): track 0.00 -> 11.9 mm
- net +5V: track 16.5 -> 19.0 mm, vias 4 -> 8
- net +BATT: track 4.74 -> 7.06 mm, vias 9 -> 14
- net Net-(C7-Pad1): track 3.07 -> 4.69 mm
- net +3.3V: track 28.4 -> 30.0 mm, vias 12 -> 13
- net /Alimentation/led_power5: track 0.00 -> 1.44 mm
- net /Alimentation/led_powerBATT: track 0.00 -> 1.31 mm
- net SWDIO: track 35.0 -> 35.7 mm
- net /SENSORS/CB_IN: track 38.2 -> 37.5 mm
- net GND: track 53.5 -> 54.0 mm, vias 86 -> 95
Other:
- board text added: "ESE2425_BAHL"

Commit message: Commit midif pcb 23/10 0816
Parts:
- added JP1: SolderJumper_2_Open, Jumper:SolderJumper-2_P1.3mm_Open_RoundedPad1.0x1.5mm, F.Cu at (138.1, 78.0)
- added JP2: SolderJumper_2_Open, Jumper:SolderJumper-2_P1.3mm_Open_RoundedPad1.0x1.5mm, F.Cu at (141.1, 78.5)
Connections:
- J7 pad 13: RX_SWD -> Net-(J7-VCP_RX)
- J7 pad 14: TX_SWD -> Net-(J7-VCP_TX)
Routing:
- net RX_SWD: track 41.2 -> 32.6 mm
- net Net-(J7-VCP_RX): track 0.00 -> 8.48 mm
- net TX_SWD: track 36.0 -> 31.1 mm
- net Net-(J7-VCP_TX): track 0.00 -> 3.66 mm
- net NRST: track 41.7 -> 39.6 mm
- net GND: vias 95 -> 93
