File: Schema_KICAD/ESE_AL8/ESE_AL8/ESE_AL8.kicad_pcb (KiCad board)
At the start: 4 copper layers, 54 x 57 mm, 87 parts, among them IC1 MP1475SGJ-P, J1 CB1, J2 CB2, J3 LIDAR, J4 Moteur1, J5 Moteur2, J6 Batterie, J7 Conn_ST_STDC14, J8 ECRAN, SW1 SW_c/s, SW2 ON/OFF, U1 ADXL343, U2 BUxxSD5, U3 STM32G431CBUx, U4 ZXBM5210-SP, U5 ZXBM5210-SP, Y1 16MHz

Commit message: Commit last modif 23/10/24 11:29
Parts:
- added TP8: TestPoint, TestPoint:TestPoint_Pad_D1.0mm, F.Cu at (147.2, 95.2)
Connections:
- U1 pad 9: unconnected-(U1-INT2-Pad9) -> /SENSORS/INT2_ACCELERO
- U3 pad 47: unconnected-(U3-PB9-Pad47) -> /SENSORS/INT2_ACCELERO
Routing:
- net /SENSORS/INT2_ACCELERO: track 0.00 -> 21.9 mm, vias 0 -> 2

Commit message: le bon ioc
Parts:
- added G***: LOGO, STM32:logo, B.Cu at (157.1, 93.7)
Routing:
- net GND: vias 93 -> 94

Commit message: push 26/11
Parts:
- moved G*** 1.86 mm to (155.6, 92.6)
Changed lines of the file:
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@@
 		(tags "capacitor")
 		(property "Reference" "C11"
-			(at 0 -1.43 90)
+			(at 1.14 -2.9 90)
 			(layer "F.SilkS")
 			(effects
@@
 	(footprint "STM32:logo"
 		(layer "B.Cu")
-		(at 157.09 93.71)
+		(at 155.62 92.57)
 		(property "Reference" "G***"
 			(at 0 0 0)
