File: Schema_KICAD/ESE_AL8/ESE_AL8/STM32.kicad_sch (KiCad schematic)
At the start: 25 parts, among them J7 Conn_ST_STDC14, U3 STM32G431CBUx, Y1 16MHz

Commit message: Commit last modif 23/10/24 11:29
Changed lines of the file:
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@@
-	)
-	(junction
-		(at 57.15 41.91)
-		(diameter 0)
-		(color 0 0 0 0)
 	)
 	(junction
@@
 	(wire
 		(pts
-			(xy 57.15 39.37) (xy 57.15 41.91)
-		)
-		(stroke
-			(width 0)
-			(type default)
-		)
-	)
-	(wire
-		(pts
 			(xy 60.96 41.91) (xy 69.85 41.91)
 		)
@@
 	(wire
 		(pts
-			(xy 57.15 41.91) (xy 60.96 41.91)
+			(xy 52.07 41.91) (xy 60.96 41.91)
 		)
 		(stroke
@@
 		(pts
 			(xy 60.96 49.53) (xy 60.96 52.07)
-		)
-		(stroke
-			(width 0)
-			(type default)
-		)
-	)
-	(wire
-		(pts
-			(xy 52.07 41.91) (xy 57.15 41.91)
 		)
 		(stroke
@@
 		(fields_autoplaced yes)
 		(effects
-			(font
-				(size 1.27 1.27)
-			)
-			(justify left)
-		)
-	)
-	(hierarchical_label "3.3V"
-		(shape input)
-		(at 57.15 39.37 90)
-		(fields_autoplaced yes)
-		(effects

Commit message: push 26/11
Parts:
- R10: value 20 -> 10
Changed lines of the file:
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@@
 			)
 		)
-		(property "Value" "20"
+		(property "Value" "10"
 			(at 57.658 102.87 0)
 			(effects
