File: Schema_KICAD/ESE_AL8/ESE_AL8/sensors.kicad_sch (KiCad schematic)
At the start: 17 parts, among them J1 CB1, J2 CB2, J3 LIDAR, J4 Moteur1, J5 Moteur2, SW1 SW_c/s, U1 ADXL343

Commit message: Commit midif pcb 23/10 0914
Parts:
- added TP8: TestPoint, TestPoint:TestPoint_Pad_D1.0mm, symbol Connector:TestPoint
Connections:
- net INT2_ACCELERO: now reaches U1.9 (INT2)
- net INT2_ACCELERO: now also TP8.1
- no-connect marks 4 -> 3
Changed lines of the file:
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@@
+	)
+	(junction
+		(at 214.63 71.12)
+		(diameter 0)
+		(color 0 0 0 0)
 	)
 	(junction
@@
 	)
 	(no_connect
-		(at 212.09 71.12)
-	)
-	(no_connect
 		(at 204.47 81.28)
 	)
@@
 		(pts
 			(xy 204.47 55.88) (xy 204.47 50.8)
+		)
+		(stroke
+			(width 0)
+			(type default)
+		)
+	)
+	(wire
+		(pts
+			(xy 217.17 71.12) (xy 214.63 71.12)
+		)
+		(stroke
+			(width 0)
+			(type default)
+		)
+	)
+	(wire
+		(pts
+			(xy 214.63 71.12) (xy 212.09 71.12)
 		)
 		(stroke
@@
 		)
 	)
+	(hierarchical_label "INT2_ACCELERO"
+		(shape input)
+		(at 217.17 71.12 0)
+		(fields_autoplaced yes)
+		(effects
+			(font
+				(size 1.27 1.27)
+				(bold yes)
+			)
+			(justify left)
+		)
+	)
 	(hierarchical_label "PHASE_A2"
 		(shape input)
@@
 		)
 		(property "Value" "TestPoint"
-			(at 214.884 71.374 0)
+			(at 217.932 72.898 0)
 			(effects
 				(font
@@
 					(unit 1)
 				)
+			)
+		)
+	)
+	(symbol
+		(lib_id "Connector:TestPoint")
+		(at 214.63 71.12 180)
+		(unit 1)
+		(exclude_from_sim no)
+		(in_bom yes)
+		(on_board yes)
+		(dnp no)
+		(property "Reference" "TP8"
+			(at 213.36 76.454 0)
+			(effects
+				(font
+					(size 1.27 1.27)
+				)
+				(justify left)
+			)
+		)
+		(property "Value" "TestPoint"
+			(at 223.266 76.708 0)
+			(effects
+				(font
+					(size 1.27 1.27)
+				)
+				(justify left)
+			)
+		)
+		(property "Footprint" "TestPoint:TestPoint_Pad_D1.0mm"
+			(at 209.55 71.12 0)
+			(effects
+				(font
+					(size 1.27 1.27)
+				)
+				(hide yes)
+			)
+		)
+		(property "Datasheet" "~"
+			(at 209.55 71.12 0)
+			(effects
+				(font
+					(size 1.27 1.27)
+				)
+				(hide yes)
+			)
+		)
+		(property "Description" "test point"
+			(at 214.63 71.12 0)
+			(effects
+				(font
+					(size 1.27 1.27)
+				)
+				(hide yes)
+			)
+		)
+		(pin "1"
+		)
+		(instances
+			(project "ESE_AL8"
+				(path "/c3d0eb52-cd9d-4e69-bcf7-3f0716f715c6/ec07ab64-4612-44cf-8e70-ea693fb6c5ed"
+					(reference "TP8")
+					(unit 1)
+				)
